File: circuit-boards/Orin-NX-PCBs/NX-J401-Adapter-v2/fan-control.kicad_sch (KiCad schematic)
At the start: 25 parts, among them J3 I2C, J7 TEMP, U2 EMC2101-R, U3 AT24CS02-SSHM, U5 ISP762T, U5 MIC5233-3.3YS

Commit message: Modified to expand M.2 adapter space, temp sensor connector and pwr LED
Signed-off-by: Scott <sgberman1@gmail.com>
Parts:
- J7: footprint NX-J401-Adapter:70541-0001 -> Connector_JST:JST_SH_BM02B-SRSS-TB_1x02-1MP_P1.00mm_Vertical; DIST P/N WM14047-ND -> 455-1788-1-ND; MFG Molex -> JST; MFG P/N 0705410001 -> BM02B-SRSS-TB
Changed lines of the file:
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@@
+    )
+  )
+  (symbol (lib_id "Graphic:SYM_Arrow_Large") (at 44.45 200.66 0) (unit 1)
+    (in_bom yes) (on_board no) (dnp no)
+    (property "Reference" "#SYM12" (at 41.91 199.39 0)
+      (effects (font (size 1.27 1.27)))
+    )
+    (property "Value" "2N3904 Transistor Temp Sensor" (at 49.53 200.66 0)
+      (effects (font (size 2.54 2.54)) (justify left))
+    )
+    (property "Footprint" "" (at 44.45 200.66 0)
+      (effects (font (size 1.27 1.27)) hide)
+    )
+    (property "Datasheet" "Components/onsemi-PZT3904-D.pdf" (at 44.45 200.66 0)
+      (effects (font (size 1.27 1.27)) hide)
+    )
+    (property "MFG" "onsemi" (at 44.45 200.66 0)
+      (effects (font (size 1.27 1.27)) hide)
+    )
+    (property "MFG P/N" "2N3904BU" (at 44.45 200.66 0)
+      (effects (font (size 1.27 1.27)) hide)
+    )
+    (property "DIST" "Digikey" (at 44.45 200.66 0)
+      (effects (font (size 1.27 1.27)) hide)
+    )
+    (property "DIST P/N" "2N3904FS-ND" (at 44.45 200.66 0)
+      (effects (font (size 1.27 1.27)) hide)
+    )
+    (instances
+      (project "NX-J401-Adapter"
+        (path "/cc31ce4b-09ab-4aea-a1d3-ed84696ba658"
+          (reference "#SYM12") (unit 1)
+        )
+        (path "/cc31ce4b-09ab-4aea-a1d3-ed84696ba658/31806f24-7fa6-46e2-ae93-f7306b662757"
+          (reference "Q3") (unit 1)
+        )
+      )
     )
   )
@@
       (effects (font (size 1.27 1.27)) (justify right))
     )
-    (property "Footprint" "NX-J401-Adapter:70541-0001" (at 111.76 154.94 0)
-      (effects (font (size 1.27 1.27)) hide)
-    )
-    (property "Datasheet" "Components/Molex-70541-0001.pdf" (at 111.76 154.94 0)
-      (effects (font (size 1.27 1.27)) hide)
-    )
-    (property "MFG" "Molex" (at 111.76 154.94 0)
-      (effects (font (size 1.27 1.27)) hide)
-    )
-    (property "MFG P/N" "0705410001" (at 111.76 154.94 0)
+    (property "Footprint" "Connector_JST:JST_SH_BM02B-SRSS-TB_1x02-1MP_P1.00mm_Vertical" (at 111.76 154.94 0)
+      (effects (font (size 1.27 1.27)) hide)
+    )
+    (property "Datasheet" "Components/JST-eSH.pdf" (at 111.76 154.94 0)
+      (effects (font (size 1.27 1.27)) hide)
+    )
+    (property "MFG" "JST" (at 111.76 154.94 0)
+      (effects (font (size 1.27 1.27)) hide)
+    )
+    (property "MFG P/N" "BM02B-SRSS-TB" (at 111.76 154.94 0)
       (effects (font (size 1.27 1.27)) hide)
     )
@@
       (effects (font (size 1.27 1.27)) hide)
     )
-    (property "DIST P/N" "WM14047-ND" (at 111.76 154.94 0)
+    (property "DIST P/N" "455-1788-1-ND" (at 111.76 154.94 0)
       (effects (font (size 1.27 1.27)) hide)
     )
@@
         )
       )
+    )
+  )
+  (symbol (lib_id "Graphic:SYM_Arrow_Large") (at 44.45 195.58 0) (unit 1)
+    (in_bom yes) (on_board no) (dnp no)
+    (property "Reference" "#SYM12" (at 41.91 194.31 0)
+      (effects (font (size 1.27 1.27)))
+    )
+    (property "Value" "JST 02SR-3S Diode Harness" (at 49.53 195.58 0)
+      (effects (font (size 2.54 2.54)) (justify left))
+    )
+    (property "Footprint" "" (at 44.45 195.58 0)
+      (effects (font (size 1.27 1.27)) hide)
+    )
+    (property "Datasheet" "https://www.digikey.com/en/products/detail/jst-sales-america-inc/A02SR02SR30K254A/9922173" (at 44.45 195.58 0)
+      (effects (font (size 1.27 1.27)) hide)
+    )
+    (property "MFG" "JST Sales" (at 44.45 195.58 0)
+      (effects (font (size 1.27 1.27)) hide)
+    )
+    (property "MFG P/N" "A02SR02SR30K254A" (at 44.45 195.58 0)
+      (effects (font (size 1.27 1.27)) hide)
+    )
+    (property "DIST" "Digikey" (at 44.45 195.58 0)
+      (effects (font (size 1.27 1.27)) hide)
+    )
+    (property "DIST P/N" "455-3623-ND" (at 44.45 195.58 0)
+      (effects (font (size 1.27 1.27)) hide)
+    )
+    (instances
+      (project "NX-J401-Adapter"
+        (path "/cc31ce4b-09ab-4aea-a1d3-ed84696ba658"
+          (reference "#SYM12") (unit 1)
+        )
+        (path "/cc31ce4b-09ab-4aea-a1d3-ed84696ba658/31806f24-7fa6-46e2-ae93-f7306b662757"
+          (reference "W1") (unit 1)
+        )
+      )
