File: circuit-boards/connector_boards/kraken-can-adapter/kraken-can-adapter.kicad_pcb (KiCad board)
At the start: 2 copper layers, 44.3 x 21.7 mm, 4 parts, among them J1 CAN, J2 CAN, J3 CAN_L, J4 CAN_H

Commit message: Increased board area to allow room for VHB between can and power boards.
Signed-off-by: Scott <sgberman1@gmail.com>
Other:
- outline, holes or cut-outs redrawn
- board text added: "H L"
