File: circuit-boards/IMU-2X-v3/LED.kicad_sch (KiCad schematic)
At the start: 14 parts, among them U11 SN74LVC2G04DBVR, U4 SN74LVC2G04DBVR

Commit message: Added some part numbers
Signed-off-by: Scott Berman <sgberman1@gmail.com>
Parts:
- renumbered C38 to C13, C38 to C44, D3 to D6, D3 to D7, R23 to R10, R23 to R24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
