File: circuit-boards/IMU-2X-v3/power-supply.kicad_sch (KiCad schematic)
At the start: 21 parts, among them U3 TPS613222ADBVR, U9 LMR54410FDBVR

Commit message: Added some part numbers
Signed-off-by: Scott Berman <sgberman1@gmail.com>
Parts:
- gave numbers to parts that had none: 3
Changed lines of the file:
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@@
   (symbol (lib_id "Device:C") (at 240.03 170.18 0) (unit 1)
     (in_bom yes) (on_board yes) (dnp no)
-    (property "Reference" "C?" (at 238.76 167.64 0)
+    (property "Reference" "C2" (at 238.76 167.64 0)
       (effects (font (size 1.27 1.27)) (justify right))
     )
@@
     (instances
       (project "IMU-2X"
-        (path "/3a012c22-a9cb-4cb7-8e69-db8529c53ea6"
-          (reference "C?") (unit 1)
-        )
         (path "/3a012c22-a9cb-4cb7-8e69-db8529c53ea6/dfddfc9c-e803-47e7-ad6c-6304a5151d35"
           (reference "C2") (unit 1)
@@
   (symbol (lib_id "Device:C") (at 227.33 170.18 0) (unit 1)
     (in_bom yes) (on_board yes) (dnp no)
-    (property "Reference" "C?" (at 226.06 167.64 0)
+    (property "Reference" "C11" (at 226.06 167.64 0)
       (effects (font (size 1.27 1.27)) (justify right))
     )
@@
     (instances
       (project "IMU-2X"
-        (path "/3a012c22-a9cb-4cb7-8e69-db8529c53ea6"
-          (reference "C?") (unit 1)
-        )
         (path "/3a012c22-a9cb-4cb7-8e69-db8529c53ea6/dfddfc9c-e803-47e7-ad6c-6304a5151d35"
           (reference "C11") (unit 1)
@@
   (symbol (lib_id "Device:C") (at 243.84 59.69 0) (unit 1)
     (in_bom yes) (on_board yes) (dnp no)
-    (property "Reference" "C?" (at 242.57 57.15 0)
+    (property "Reference" "C7" (at 242.57 57.15 0)
       (effects (font (size 1.27 1.27)) (justify right))
     )
@@
     (instances
       (project "IMU-2X"
-        (path "/3a012c22-a9cb-4cb7-8e69-db8529c53ea6"
-          (reference "C?") (unit 1)
-        )
         (path "/3a012c22-a9cb-4cb7-8e69-db8529c53ea6/dfddfc9c-e803-47e7-ad6c-6304a5151d35"
           (reference "C7") (unit 1)
