File: circuit-boards/IMU-2X-v3/pwm-heading.kicad_sch (KiCad schematic)
At the start: 9 parts, among them J9 HEADING, J9 RATE, U13 ISO6720FBDR

Commit message: Added some part numbers
Signed-off-by: Scott Berman <sgberman1@gmail.com>
Parts:
- C41, C42: renamed from C31; DIST (none) -> Digikey; DIST P/N (none) -> 399-C1206C104K3RAC7800CT-ND; MFG (none) -> KEMET; MFG P/N (none) -> C1206C104K3RAC7800
- renumbered D2 to D4, D2 to D5, R21 to R19, R21 to R23
Changed lines of the file:
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@@
   (symbol (lib_id "Device:C") (at 156.21 92.71 0) (mirror y) (unit 1)
     (in_bom yes) (on_board yes) (dnp no)
-    (property "Reference" "C31" (at 152.4 92.71 0)
+    (property "Reference" "C41" (at 152.4 92.71 0)
       (effects (font (size 1.27 1.27)) (justify left))
     )
@@
       (effects (font (size 1.27 1.27)) hide)
     )
-    (property "Datasheet" "" (at 156.21 92.71 0)
-      (effects (font (size 1.27 1.27)) hide)
-    )
-    (property "DIST" "" (at 156.21 92.71 0)
-      (effects (font (size 1.27 1.27)) hide)
-    )
-    (property "DIST P/N" "" (at 156.21 92.71 0)
-      (effects (font (size 1.27 1.27)) hide)
-    )
-    (property "MFG" "" (at 156.21 92.71 0)
-      (effects (font (size 1.27 1.27)) hide)
-    )
-    (property "MFG P/N" "" (at 156.21 92.71 0)
-      (effects (font (size 1.27 1.27)) hide)
-    )
-    (pin "1")
-    (pin "2")
-    (instances
-      (project "IMU-2X"
-        (path "/3a012c22-a9cb-4cb7-8e69-db8529c53ea6"
-          (reference "C31") (unit 1)
-        )
+    (property "Datasheet" "https://www.digikey.com/en/products/detail/kemet/C1206C104K3RAC7800/2215076" (at 156.21 92.71 0)
+      (effects (font (size 1.27 1.27)) hide)
+    )
+    (property "DIST" "Digikey" (at 156.21 92.71 0)
+      (effects (font (size 1.27 1.27)) hide)
+    )
+    (property "DIST P/N" "399-C1206C104K3RAC7800CT-ND" (at 156.21 92.71 0)
+      (effects (font (size 1.27 1.27)) hide)
+    )
+    (property "MFG" "KEMET" (at 156.21 92.71 0)
+      (effects (font (size 1.27 1.27)) hide)
+    )
+    (property "MFG P/N" "C1206C104K3RAC7800" (at 156.21 92.71 0)
+      (effects (font (size 1.27 1.27)) hide)
+    )
+    (pin "1")
+    (pin "2")
+    (instances
+      (project "IMU-2X"
         (path "/3a012c22-a9cb-4cb7-8e69-db8529c53ea6/4bacb90b-5ef0-490f-9fcc-20f01791f70e"
           (reference "C41") (unit 1)
@@
   (symbol (lib_id "power:+3V3") (at 163.83 104.14 0) (unit 1)
     (in_bom yes) (on_board yes) (dnp no)
-    (property "Reference" "#PWR037" (at 163.83 107.95 0)
+    (property "Reference" "#PWR090" (at 163.83 107.95 0)
       (effects (font (size 1.27 1.27)) hide)
     )
@@
     (instances
       (project "IMU-2X"
-        (path "/3a012c22-a9cb-4cb7-8e69-db8529c53ea6"
-          (reference "#PWR037") (unit 1)
-        )
         (path "/3a012c22-a9cb-4cb7-8e69-db8529c53ea6/4bacb90b-5ef0-490f-9fcc-20f01791f70e"
           (reference "#PWR090") (unit 1)
@@
   (symbol (lib_id "Device:D_Schottky") (at 212.09 77.47 0) (mirror x) (unit 1)
     (in_bom yes) (on_board yes) (dnp no)
-    (property "Reference" "D2" (at 212.09 72.39 0)
+    (property "Reference" "D4" (at 212.09 72.39 0)
       (effects (font (size 1.27 1.27)))
     )
@@
     (instances
       (project "IMU-2X"
-        (path "/3a012c22-a9cb-4cb7-8e69-db8529c53ea6/dfddfc9c-e803-47e7-ad6c-6304a5151d35"
-          (reference "D2") (unit 1)
-        )
         (path "/3a012c22-a9cb-4cb7-8e69-db8529c53ea6/4bacb90b-5ef0-490f-9fcc-20f01791f70e"
           (reference "D4") (unit 1)
@@
   (symbol (lib_id "Device:D_Schottky") (at 212.09 86.36 0) (mirror x) (unit 1)
     (in_bom yes) (on_board yes) (dnp no)
-    (property "Reference" "D2" (at 212.09 81.28 0)
+    (property "Reference" "D5" (at 212.09 81.28 0)
       (effects (font (size 1.27 1.27)))
     )
@@
     (instances
       (project "IMU-2X"
-        (path "/3a012c22-a9cb-4cb7-8e69-db8529c53ea6/dfddfc9c-e803-47e7-ad6c-6304a5151d35"
-          (reference "D2") (unit 1)
-        )
         (path "/3a012c22-a9cb-4cb7-8e69-db8529c53ea6/4bacb90b-5ef0-490f-9fcc-20f01791f70e"
           (reference "D5") (unit 1)
@@
   (symbol (lib_id "Device:C") (at 194.31 92.71 0) (unit 1)
     (in_bom yes) (on_board yes) (dnp no)
-    (property "Reference" "C31" (at 198.12 92.71 0)
+    (property "Reference" "C42" (at 198.12 92.71 0)
       (effects (font (size 1.27 1.27)) (justify left))
     )
@@
       (effects (font (size 1.27 1.27)) hide)
     )
-    (property "Datasheet" "" (at 194.31 92.71 0)
-      (effects (font (size 1.27 1.27)) hide)
-    )
-    (property "DIST" "" (at 194.31 92.71 0)
-      (effects (font (size 1.27 1.27)) hide)
-    )
-    (property "DIST P/N" "" (at 194.31 92.71 0)
-      (effects (font (size 1.27 1.27)) hide)
-    )
-    (property "MFG" "" (at 194.31 92.71 0)
-      (effects (font (size 1.27 1.27)) hide)
-    )
-    (property "MFG P/N" "" (at 194.31 92.71 0)
-      (effects (font (size 1.27 1.27)) hide)
-    )
-    (pin "1")
-    (pin "2")
-    (instances
-      (project "IMU-2X"
-        (path "/3a012c22-a9cb-4cb7-8e69-db8529c53ea6"
-          (reference "C31") (unit 1)
-        )
+    (property "Datasheet" "https://www.digikey.com/en/products/detail/kemet/C1206C104K3RAC7800/2215076" (at 194.31 92.71 0)
+      (effects (font (size 1.27 1.27)) hide)
+    )
+    (property "DIST" "Digikey" (at 194.31 92.71 0)
+      (effects (font (size 1.27 1.27)) hide)
+    )
+    (property "DIST P/N" "399-C1206C104K3RAC7800CT-ND" (at 194.31 92.71 0)
+      (effects (font (size 1.27 1.27)) hide)
+    )
+    (property "MFG" "KEMET" (at 194.31 92.71 0)
+      (effects (font (size 1.27 1.27)) hide)
+    )
+    (property "MFG P/N" "C1206C104K3RAC7800" (at 194.31 92.71 0)
+      (effects (font (size 1.27 1.27)) hide)
+    )
+    (pin "1")
+    (pin "2")
+    (instances
+      (project "IMU-2X"
         (path "/3a012c22-a9cb-4cb7-8e69-db8529c53ea6/4bacb90b-5ef0-490f-9fcc-20f01791f70e"
           (reference "C42") (unit 1)
@@
   (symbol (lib_id "Device:R_US") (at 200.66 119.38 270) (mirror x) (unit 1)
     (in_bom yes) (on_board yes) (dnp no)
-    (property "Reference" "R21" (at 200.66 116.84 90)
+    (property "Reference" "R23" (at 200.66 116.84 90)
       (effects (font (size 1.27 1.27)))
     )
@@
     (instances
       (project "IMU-2X"
-        (path "/3a012c22-a9cb-4cb7-8e69-db8529c53ea6"
-          (reference "R21") (unit 1)
-        )
-        (path "/3a012c22-a9cb-4cb7-8e69-db8529c53ea6/088575d8-b480-483a-8195-b5bd2af558b0"
-          (reference "R20") (unit 1)
-        )
         (path "/3a012c22-a9cb-4cb7-8e69-db8529c53ea6/4bacb90b-5ef0-490f-9fcc-20f01791f70e"
           (reference "R23") (unit 1)
@@
   (symbol (lib_id "Device:R_US") (at 200.66 109.22 270) (mirror x) (unit 1)
     (in_bom yes) (on_board yes) (dnp no)
-    (property "Reference" "R21" (at 200.66 106.68 90)
+    (property "Reference" "R19" (at 200.66 106.68 90)
       (effects (font (size 1.27 1.27)))
     )
@@
     (instances
       (project "IMU-2X"
-        (path "/3a012c22-a9cb-4cb7-8e69-db8529c53ea6"
-          (reference "R21") (unit 1)
-        )
-        (path "/3a012c22-a9cb-4cb7-8e69-db8529c53ea6/088575d8-b480-483a-8195-b5bd2af558b0"
-          (reference "R20") (unit 1)
-        )
         (path "/3a012c22-a9cb-4cb7-8e69-db8529c53ea6/4bacb90b-5ef0-490f-9fcc-20f01791f70e"
           (reference "R19") (unit 1)
@@
   (symbol (lib_id "power:GND") (at 156.21 96.52 0) (unit 1)
     (in_bom yes) (on_board yes) (dnp no)
-    (property "Reference" "#PWR035" (at 156.21 102.87 0)
+    (property "Reference" "#PWR089" (at 156.21 102.87 0)
       (effects (font (size 1.27 1.27)) hide)
     )
@@
     (instances
       (project "IMU-2X"
-        (path "/3a012c22-a9cb-4cb7-8e69-db8529c53ea6"
-          (reference "#PWR035") (unit 1)
-        )
         (path "/3a012c22-a9cb-4cb7-8e69-db8529c53ea6/4bacb90b-5ef0-490f-9fcc-20f01791f70e"
           (reference "#PWR089") (unit 1)
@@
   (symbol (lib_id "power:GND") (at 163.83 124.46 0) (unit 1)
     (in_bom yes) (on_board yes) (dnp no)
-    (property "Reference" "#PWR035" (at 163.83 130.81 0)
+    (property "Reference" "#PWR091" (at 163.83 130.81 0)
       (effects (font (size 1.27 1.27)) hide)
     )
@@
     (instances
       (project "IMU-2X"
-        (path "/3a012c22-a9cb-4cb7-8e69-db8529c53ea6"
-          (reference "#PWR035") (unit 1)
-        )
         (path "/3a012c22-a9cb-4cb7-8e69-db8529c53ea6/4bacb90b-5ef0-490f-9fcc-20f01791f70e"
           (reference "#PWR091") (unit 1)
@@
   (symbol (lib_id "power:+3V3") (at 156.21 88.9 0) (unit 1)
     (in_bom yes) (on_board yes) (dnp no)
-    (property "Reference" "#PWR037" (at 156.21 92.71 0)
+    (property "Reference" "#PWR088" (at 156.21 92.71 0)
       (effects (font (size 1.27 1.27)) hide)
     )
@@
     (instances
       (project "IMU-2X"
-        (path "/3a012c22-a9cb-4cb7-8e69-db8529c53ea6"
-          (reference "#PWR037") (unit 1)
-        )
         (path "/3a012c22-a9cb-4cb7-8e69-db8529c53ea6/4bacb90b-5ef0-490f-9fcc-20f01791f70e"
           (reference "#PWR088") (unit 1)
