File: circuit-boards/connector_boards/MAG_encoder_adapter/MAG_encoder_adapter.kicad_sch (KiCad schematic)
At the start: 5 parts, among them J1 Mag-encoder, J2 POT, J3 RIO

Commit message: Updated boms and exported output files for connector boards
Signed-off-by: Scott <sgberman1@gmail.com>
Parts:
- D1: DIST (none) -> Digikey; DIST P/N (none) -> 1080-1419-1-ND; MFG (none) -> Everlight Electronics Co Ltd; MFG P/N (none) -> QTLP650D4TR
- J1: DIST (none) -> Digikey; DIST P/N (none) -> 609-4054-ND
- J2: DIST (none) -> Digikey; DIST P/N (none) -> WM4165-ND; MFG MOLEX -> Molex
- J3: DIST (none) -> Digikey; DIST P/N (none) -> 23-0705550005-ND; MFG (none) -> Molex; MFG P/N (none) -> 705550005
- R1: DIST (none) -> Digikey; DIST P/N (none) -> 311-2.0KARCT-ND; MFG (none) -> YAGEO; MFG P/N (none) -> RC0805JR-072KL
