File: circuit-boards/connector_boards/potentiometer_adapter/potentiometer_adapter.kicad_sch (KiCad schematic)
At the start: 4 parts, among them J1 Conn_01x03_Male

Commit message: Updated boms and exported output files for connector boards
Signed-off-by: Scott <sgberman1@gmail.com>
Parts:
- D1: DIST (none) -> Digikey; DIST P/N (none) -> 1080-1419-1-ND; MFG (none) -> Everlight Electronics Co Ltd; MFG P/N (none) -> QTLP650D4TR
- J1: DIST (none) -> Digikey; DIST P/N (none) -> WM20415-ND; MFG (none) -> Molex; MFG P/N (none) -> 0705410037
- R1: DIST (none) -> Digikey; DIST P/N (none) -> 311-2.0KARCT-ND; MFG (none) -> YAGEO; MFG P/N (none) -> RC0805JR-072KL
- RV1: MFG (none) -> Bourns
