File: robots/2024/system-drawing/kicad-schematic/2024-SystemDiagram.kicad_sch (KiCad schematic)
At the start: 166 parts

Commit message: Add PD fuse and Orin NX symbols
Signed-off-by: Scott Berman <sgberman1@gmail.com>
Parts:
- added A1: Orin NX1, symbol SystemDiagram:Orin_NX
- added A2: Orin NX2, symbol SystemDiagram:Orin_NX
- added A3: Orin NX3, symbol SystemDiagram:Orin_NX
- added F1, F2, F3, F4, F5: 10A, symbol SystemDiagram:Circuit_Breaker
- added PD2: PDF, symbol SystemDiagram:Power_Distribution_-_Fuse
Connections:
- net at WG15. (2): now also W27.1; no longer W60.1
- net at W27.1: no longer WG15. (2)
- net at VRM1. (5V/2A): now also W54.1
- net at POE?. (RJ45S): now also W45.1; no longer VRM1. (5V/2A)
- net at W54.1: now also RDO1. (POWER); no longer VRM1. (5V/2A)
- net at MGA1. (POT): now also W18.1; no longer W13.1
- net at WG6. (4): now also FAN1.1 (+); no longer W68.1
- net at W19.1: now also MAG2. (OUT); no longer MGA2. (POT)
- net at W56.1: now also IND1. (P); no longer WG5. (3)
- net at WG3. (5): now also W27.1; no longer WG5. (3)
- net at MOT3. (PWR): no longer MOT2. (PWR)
- net at W62.1: now also W36.1; no longer MOT10. (PWR)
- net at W36.1: now also MOT6. (PWR); no longer W62.1
- net at W52.1: now also ETH1. (POWER); no longer RDO1. (POWER)
- net at IMU1. (RIO_PWM): now also W12.1; no longer W33.1
- net at CB1.CB: now also W3.1; no longer W1.1
- net at W3.1: now also PD1.VIN_POS; no longer CB1.CB
- net at MGA4. (POT): now also W24.1; no longer W65.1
- net at W23.1: now also MAG4. (OUT); no longer MGA4. (POT)
- net at W24.1: now also POT4. (OUT); no longer MGA4. (POT)
- net at BBA3. (SNSR): now also W38.1
- net at W60.1: now also WG3. (5); no longer BBA3. (SNSR)
- net at WG2. (5): now also W27.1
- net at W59.1: now also WG3. (5); no longer WG2. (5)
- net at W42.1: now also CAM1.; no longer PI3. (USB3)
- net at W11.1: now also ENCA1. (OUT); no longer IMU1. (RIO_PWM)
- net at ENCA1. (OUT): now also ENC1. (OUT); no longer W11.1
- net at WG8. (3): now also FAN3.1 (+); no longer W73.1
- net at WG9. (3): now also FAN3.2 (-); no longer W73.1
- net at VRM2. (5V/2A): no longer W25.1
- net at WG10. (4): now also FAN2.1 (+); no longer W71.1
- net at WG11. (4): now also FAN2.2 (-); no longer W71.1
- net at W47.1: now also ETH1. (POWER); no longer PI3. (USB3)
- net at W46.1: now also PI2. (USB3); no longer ETH1. (POWER)
- net at W50.1: now also PI6. (USB3); no longer ETH1. (POWER)
- net at W48.1: now also PI4. (USB3); no longer ETH1. (POWER)
- net at W51.1: now also PI1. (USB3); no longer ETH1. (POWER)
- net at W49.1: now also PI5. (USB3); no longer ETH1. (POWER)
- net at WG7. (4): now also FAN1.2 (-); no longer W68.1
- net at W18.1: now also POT1. (OUT); no longer MGA1. (POT)
- net at W30.1: now also PI1. (USB3); no longer IMU1. (RIO_PWM)
- net at PI1. (USB3): no longer W30.1
- net at IND1. (P): now also W61.1; no longer W56.1
- net at PI6. (USB3): no longer W50.1
- net at MGA2. (POT): now also W14.1; no longer W20.1
- net at W31.1: now also W27.1; no longer TFC1. (OUT)
- net at W64.1: now also MGA3. (POT); no longer W15.1
- net at BBA2. (SNSR): now also W59.1
- net at W66.1: now also PI6. (USB3); no longer WG8. (3)
- net at WG16. (2): now also W27.1; no longer W59.1
- net LEFT_UNDER_DRIVE_PWR: no longer names the net of PD1.T2
- net LEFT_UNDER_DRIVE_PWR: no longer MOT3. (PWR)
- net RIGHT_UNDER_DRIVE_PWR: no longer names the net of PD1.T15
- net RIGHT_UNDER_DRIVE_PWR: no longer MOT6. (PWR)
- new net: W60.1, WG15. (2)
- new net: POE?. (RJ45S), VRM1. (5V/2A)
- new net: VRM1. (5V/2A), W53.1
- new net: MGA1. (POT), W13.1
- new net: W68.1, WG6. (4)
- new net: W67.1, WG6. (4)
- new net: W69.1, WG6. (4)
- new net: MGA2. (POT), W19.1
- new net: MOT8. (PWR), W58.1
- new net: POE?. (RJ45S), RDO1. (POWER)
- new net: W56.1, WG5. (3)
- new net: WG3. (5), WG5. (3)
- new net: MOT1. (PWR), MOT2. (PWR)
- new net: MOT2. (PWR), MOT3. (PWR)
- new net: MOT10. (PWR), W62.1
- new net: RDO1. (POWER), W52.1
- new net: IMU1. (RIO_PWM), W33.1
- new net: CB1.CB, W1.1
- new net: MGA4. (POT), W65.1
- new net: MGA4. (POT), W23.1
- new net: F1.CB, PD2. (IN)
- new net: BBA3. (SNSR), W60.1
- new net: WG2. (5), WG4. (3)
- new net: W60.1, WG2. (5)
- new net: W59.1, WG2. (5)
- new net: PI3. (USB3), W42.1
- new net: IMU1. (RIO_PWM), W11.1
- new net: W73.1, WG8. (3)
- new net: W73.1, WG9. (3)
- new net: IMU1. (RIO_PWM), W35.1
- new net: VRM2. (5V/2A), W25.1
- new net: MOT5. (PWR), MOT6. (PWR)
- new net: W71.1, WG10. (4)
- new net: W71.1, WG11. (4)
- new net: PI3. (USB3), W47.1
- new net: MOT3. (PWR), MOT4. (PWR)
- new net: MOT4. (PWR), MOT5. (PWR)
- new net: ETH1. (POWER), W46.1
- new net: ETH1. (POWER), W50.1
- new net: ETH1. (POWER), W48.1
- new net: ETH1. (POWER), W51.1
- new net: ETH1. (POWER), W49.1
- new net: VRM2. (5V/2A), W32.1
- new net: W68.1, WG7. (4)
- new net: W27.1, WG1. (2)
- new net: VRM2. (5V/2A), W39.1
- new net: F3.CB, PD2. (IN)
- new net: F4.CB, PD2. (IN)
- new net: F2.CB, PD2. (IN)
- new net: F5.CB, PD2. (IN)
- new net: W67.1, WG7. (4)
- new net: IMU1. (RIO_PWM), W30.1
- new net: W56.1, WG4. (3)
- new net: W70.1, WG10. (4)
- new net: W70.1, WG11. (4)
- new net: IMU1. (RIO_PWM), W34.1
- new net: MGA2. (POT), W20.1
- new net: TFC1. (OUT), W31.1
- new net: W63.1, WG10. (4)
- new net: W15.1, W64.1
- new net: BBA2. (SNSR), W37.1
- new net: VRM2. (5V/2A), W26.1
- new net: W66.1, WG8. (3)
- new net: W66.1, WG9. (3)
- new net: MOT7. (PWR), W57.1
- new net: W63.1, WG11. (4)
- new net: W59.1, WG16. (2)
- new net: W69.1, WG7. (4)
- new net: PI1. (USB3), W74.1
- now unconnected: MOT3. (PWR), PI1. (USB3), PI1. (USB3), PI6. (USB3), VRM2. (5V/2A), VRM2. (5V/2A), VRM2. (5V/2A), W27.1, W27.1, W27.1, W27.1, W27.1

Commit message: Add wire tag to use instead of cable symbol.
Signed-off-by: Scott <sgberman1@gmail.com>
Parts:
- added LINK: 2024 Wire List Link, symbol Graphic:SYM_Arrow_Large
- added W55: IMU:ENC1-ENCA1, symbol SystemDiagram:WireTag
Connections:
- net at WG15. (2): now also W27.1; no longer W60.1
- net at W27.1: no longer WG15. (2)
- net at VRM1. (5V/2A): now also W54.1
- net at POE?. (RJ45S): now also W45.1; no longer VRM1. (5V/2A)
- net at W54.1: now also RDO1. (POWER); no longer VRM1. (5V/2A)
- net at MGA1. (POT): now also W18.1; no longer W13.1
- net at WG6. (4): now also FAN1.1 (+); no longer W68.1
- net at W19.1: now also MAG2. (OUT); no longer MGA2. (POT)
- net at W56.1: now also IND1. (P); no longer WG5. (3)
- net at WG3. (5): now also W27.1; no longer WG5. (3)
- net at MOT3. (PWR): no longer MOT2. (PWR)
- net at W62.1: now also W36.1; no longer MOT10. (PWR)
- net at W36.1: now also MOT6. (PWR); no longer W62.1
- net at W52.1: now also ETH1. (POWER); no longer RDO1. (POWER)
- net at IMU1. (RIO_PWM): now also W12.1; no longer W33.1
- net at CB1.CB: now also W3.1; no longer W1.1
- net at W3.1: now also PD1.VIN_POS; no longer CB1.CB
- net at MGA4. (POT): now also W24.1; no longer W65.1
- net at W23.1: now also MAG4. (OUT); no longer MGA4. (POT)
- net at W24.1: now also POT4. (OUT); no longer MGA4. (POT)
- net at BBA3. (SNSR): now also W38.1
- net at W60.1: now also WG3. (5); no longer BBA3. (SNSR)
- net at WG2. (5): now also W27.1
- net at W59.1: now also WG3. (5); no longer WG2. (5)
- net at W42.1: now also CAM1.; no longer PI3. (USB3)
- net at W11.1: now also ENCA1. (OUT); no longer IMU1. (RIO_PWM)
- net at ENCA1. (OUT): now also ENC1. (OUT); no longer W11.1
- net at WG8. (3): now also FAN3.1 (+); no longer W73.1
- net at WG9. (3): now also FAN3.2 (-); no longer W73.1
- net at VRM2. (5V/2A): no longer W25.1
- net at WG10. (4): now also FAN2.1 (+); no longer W71.1
- net at WG11. (4): now also FAN2.2 (-); no longer W71.1
- net at W47.1: now also ETH1. (POWER); no longer PI3. (USB3)
- net at W46.1: now also PI2. (USB3); no longer ETH1. (POWER)
- net at W50.1: now also PI6. (USB3); no longer ETH1. (POWER)
- net at W48.1: now also PI4. (USB3); no longer ETH1. (POWER)
- net at W51.1: now also PI1. (USB3); no longer ETH1. (POWER)
- net at W49.1: now also PI5. (USB3); no longer ETH1. (POWER)
- net at WG7. (4): now also FAN1.2 (-); no longer W68.1
- net at PD2. (IN): now also F5.CB
- net at W18.1: now also POT1. (OUT); no longer MGA1. (POT)
- net at W30.1: now also PI1. (USB3); no longer IMU1. (RIO_PWM)
- net at PI1. (USB3): no longer W30.1
- net at IND1. (P): now also W61.1; no longer W56.1
- net at PI6. (USB3): no longer W50.1
- net at MGA2. (POT): now also W14.1; no longer W20.1
- net at W31.1: now also W27.1; no longer TFC1. (OUT)
- net at W64.1: now also MGA3. (POT); no longer W15.1
- net at BBA2. (SNSR): now also W59.1
- net at W66.1: now also PI6. (USB3); no longer WG8. (3)
- net at WG16. (2): now also W27.1; no longer W59.1
- new net: W60.1, WG15. (2)
- new net: POE?. (RJ45S), VRM1. (5V/2A)
- new net: VRM1. (5V/2A), W53.1
- new net: MGA1. (POT), W13.1
- new net: W68.1, WG6. (4)
- new net: W67.1, WG6. (4)
- new net: W69.1, WG6. (4)
- new net: MGA2. (POT), W19.1
- new net: MOT8. (PWR), W58.1
- new net: POE?. (RJ45S), RDO1. (POWER)
- new net: W56.1, WG5. (3)
- new net: WG3. (5), WG5. (3)
- new net: MOT1. (PWR), MOT2. (PWR)
- new net: MOT2. (PWR), MOT3. (PWR)
- new net: MOT10. (PWR), W62.1
- new net: RDO1. (POWER), W52.1
- new net: IMU1. (RIO_PWM), W33.1
- new net: CB1.CB, W1.1
- new net: MGA4. (POT), W65.1
- new net: MGA4. (POT), W23.1
- new net: BBA3. (SNSR), W60.1
- new net: WG2. (5), WG4. (3)
- new net: W60.1, WG2. (5)
- new net: W59.1, WG2. (5)
- new net: PI3. (USB3), W42.1
- new net: IMU1. (RIO_PWM), W11.1, W55.
- new net: W73.1, WG8. (3)
- new net: W73.1, WG9. (3)
- new net: IMU1. (RIO_PWM), W35.1
- new net: VRM2. (5V/2A), W25.1
- new net: MOT5. (PWR), MOT6. (PWR)
- new net: W71.1, WG10. (4)
- new net: W71.1, WG11. (4)
- new net: PI3. (USB3), W47.1
- new net: MOT3. (PWR), MOT4. (PWR)
- new net: MOT4. (PWR), MOT5. (PWR)
- new net: ETH1. (POWER), W46.1
- new net: ETH1. (POWER), W50.1
- new net: ETH1. (POWER), W48.1
- new net: ETH1. (POWER), W51.1
- new net: ETH1. (POWER), W49.1
- new net: VRM2. (5V/2A), W32.1
- new net: W68.1, WG7. (4)
- new net: W27.1, WG1. (2)
- new net: VRM2. (5V/2A), W39.1
- new net: W67.1, WG7. (4)
- new net: IMU1. (RIO_PWM), W30.1
- new net: W56.1, WG4. (3)
- new net: W70.1, WG10. (4)
- new net: W70.1, WG11. (4)
- new net: IMU1. (RIO_PWM), W34.1
- new net: MGA2. (POT), W20.1
- new net: TFC1. (OUT), W31.1
- new net: W63.1, WG10. (4)
- new net: W15.1, W64.1
- new net: BBA2. (SNSR), W37.1
- new net: VRM2. (5V/2A), W26.1
- new net: W66.1, WG8. (3)
- new net: W66.1, WG9. (3)
- new net: MOT7. (PWR), W57.1
- new net: W63.1, WG11. (4)
- new net: W59.1, WG16. (2)
- new net: W69.1, WG7. (4)
- new net: PI1. (USB3), W74.1
- now unconnected: MOT3. (PWR), PI1. (USB3), PI1. (USB3), PI6. (USB3), VRM2. (5V/2A), VRM2. (5V/2A), VRM2. (5V/2A), W27.1, W27.1, W27.1, W27.1, W27.1
Changed lines of the file:
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@@
     (company "971 Spartan Robotics")
   )
+  (junction (at 402.59 92.71) (diameter 0) (color 0 0 0 0)
+  )
   (no_connect (at 445.77 401.32))
   (no_connect (at 527.05 441.96))
@@
     (stroke (width 0) (type default))
   )
-  (wire (pts (xy 417.83 452.12) (xy 518.16 452.12))
+  (wire (pts (xy 402.59 92.71) (xy 396.24 92.71))
     (stroke (width 0) (type default))
   )
-  (wire (pts (xy 510.54 67.31) (xy 322.58 67.31))
+  (wire (pts (xy 417.83 452.12) (xy 518.16 452.12))
     (stroke (width 0) (type default))
   )
@@
     (stroke (width 0) (type default))
   )
+  (wire (pts (xy 322.58 67.31) (xy 510.54 67.31))
+    (stroke (width 0) (type default))
+  )
   (wire (pts (xy 430.53 151.13) (xy 400.05 151.13))
     (stroke (width 0) (type default))
@@
     (stroke (width 0) (type default))
   )
-  (wire (pts (xy 430.53 92.71) (xy 396.24 92.71))
+  (wire (pts (xy 430.53 92.71) (xy 402.59 92.71))
     (stroke (width 0) (type default))
   )
@@
     )
   )
+  (symbol (lib_id "SystemDiagram:WireTag") (at 402.59 92.71 0) (unit 1)
+    (in_bom yes) (on_board yes) (dnp no)
+    (property "Reference" "W55" (at 402.59 87.63 0)
+      (effects (font (size 1.27 1.27)))
+    )
+    (property "Value" "IMU:ENC1-ENCA1" (at 402.59 90.17 0)
+      (effects (font (size 1.27 1.27)))
+    )
+    (property "Footprint" "" (at 402.59 92.71 0)
+      (effects (font (size 1.27 1.27)) hide)
+    )
+    (property "Datasheet" "wires/W55.md" (at 402.59 92.71 0)
+      (effects (font (size 1.27 1.27)) hide)
+    )
+    (pin "")
+    (instances
+      (project "2024-SystemDiagram"
+        (path "/12a52703-e3f4-4774-b510-3055ab1abf35"
+          (reference "W55") (unit 1)
+        )
+      )
+    )
+  )
   (symbol (lib_name "Cable_7") (lib_id "SystemDiagram:Cable") (at 422.91 388.62 0) (unit 1)
     (in_bom yes) (on_board yes) (dnp no) (fields_autoplaced)
@@
         )
       )
+    )
+  )
+  (symbol (lib_id "Graphic:SYM_Arrow_Large") (at 303.53 535.94 0) (unit 1)
+    (in_bom no) (on_board no) (dnp no)
+    (property "Reference" "LINK" (at 303.53 533.654 0)
+      (effects (font (size 1.27 1.27)) hide)
+    )
+    (property "Value" "2024 Wire List Link" (at 308.61 535.94 0)
+      (effects (font (size 2.54 2.54) bold) (justify left))
+    )
+    (property "Footprint" "" (at 303.53 535.94 0)
+      (effects (font (size 1.27 1.27)) hide)
+    )
+    (property "Datasheet" "https://docs.google.com/spreadsheets/d/1T15qpFhWk4HCYvBFHs1Tk5gMzd4x4hG0uZYPDu6nkqc/edit#gid=0" (at 303.53 535.94 0)
+      (effects (font (size 1.27 1.27)) hide)
+    )
+    (instances
+      (project "2024-SystemDiagram"
+        (path "/12a52703-e3f4-4774-b510-3055ab1abf35"
+          (reference "LINK") (unit 1)
+        )
+      )

Commit message: Adding initial system drawing that include motors
Signed-off-by: Scott Berman <sgberman1@gmail.com>
Parts:
- removed CAM1: CAM_NW, symbol SystemDiagram:Camera
- removed CAM2: CAM_NE, symbol SystemDiagram:Camera
- removed CAM3: DRIVER CAM, symbol SystemDiagram:Camera
- removed CAM4: CAM_SE, symbol SystemDiagram:Camera
- removed CAM5: CAM_SW, symbol SystemDiagram:Camera
- removed CAN2, CAN3: CAN_Terminator, symbol SystemDiagram:CAN_Terminator
- removed ENCA1, ENCA2: EncoderAdapter, symbol SystemDiagram:EncoderAdapter
- removed ETH1: Ethernet_Switch, symbol SystemDiagram:Ethernet_Switch
- removed FAN1, FAN2: Fan, symbol Motor:Fan
- removed FAN3: DriverPI Fan, symbol Motor:Fan
- removed FAN4: IMU PI Fan, symbol Motor:Fan
- removed IMU1: IMU, symbol SystemDiagram:IMU
- removed IND1: CANdle, symbol SystemDiagram:CANdle
- removed MC1: SPX_ROLL, symbol SystemDiagram:Motor_Controller
- removed MC2: SPX_WRIST, symbol SystemDiagram:Motor_Controller
- removed MOT11: BAG_WRIST, symbol SystemDiagram:Motor_DC
- removed MOT9: BAG_ROLL, symbol SystemDiagram:Motor_DC
- removed PI1: IMU_PI, symbol SystemDiagram:RockPI
- removed PI2: NE_PI, symbol SystemDiagram:RockPI
- removed PI3: NW_PI, symbol SystemDiagram:RockPI
- removed PI4: SE_PI, symbol SystemDiagram:RockPI
- removed PI5: SW_PI, symbol SystemDiagram:RockPI
- removed PI6: DRIVER_PI, symbol SystemDiagram:RockPI
- removed TFC1: TOF_CONTROLLER, symbol SystemDiagram:TOF_CONTROLLER
- removed TOF1: TOF_LEFT, symbol SystemDiagram:TOF_Sensor
- removed TOF2: TOF_RIGHT, symbol SystemDiagram:TOF_Sensor
- removed VRM2: VRM, symbol SystemDiagram:VRM
- removed W1: BT1-CB1-4AWG-RED, symbol SystemDiagram:Cable
- removed W10: CTLR_PWR-18AWG, symbol SystemDiagram:Cable
- removed W11: IMU:ENC1-ENCA1, symbol SystemDiagram:Cable
- removed W12: IMU:ENC2-ENCA2, symbol SystemDiagram:Cable
- removed W13: ENC_AD2-MGA1, symbol SystemDiagram:Cable
- removed W14: ENC_AD3-MGA2, symbol SystemDiagram:Cable
- removed W15: ENC_AD4-W64, symbol SystemDiagram:Cable
- removed W16: ENC_AD5-W65, symbol SystemDiagram:Cable
- removed W17: MGA1-MAG1, symbol SystemDiagram:Cable
- removed W18: MGA1-POT1, symbol SystemDiagram:Cable
- removed W19: MGA2-MAG2, symbol SystemDiagram:Cable
- removed W2: BT1-PD1-4AWG-BLK, symbol SystemDiagram:Cable
- removed W20: MGA2-POT2, symbol SystemDiagram:Cable
- removed W21: MGA3-MAG3, symbol SystemDiagram:Cable
- removed W22: MGA3-POT3, symbol SystemDiagram:Cable
- removed W23: MGA4-MAG4, symbol SystemDiagram:Cable
- removed W24: MGA4-POT4, symbol SystemDiagram:Cable
- removed W25: VRM2_PWR, symbol SystemDiagram:Cable
- removed W26: VRM2:12V2A_WG2, symbol SystemDiagram:Cable
- removed W27: BBA-W31, symbol SystemDiagram:Cable16
- removed W28: TFC1:I2C1-TOF1, symbol SystemDiagram:Cable
- removed W29: TFC1:I2C2-TOF2, symbol SystemDiagram:Cable
- removed W3: CB1-PD1-4AWG-RED, symbol SystemDiagram:Cable
- removed W30: PI1:IMU-IMU1:PI_OUT, symbol SystemDiagram:Cable
- removed W31: W27-TFC1:OUT, symbol SystemDiagram:Cable
- removed W32: VRM2:5V2A_WG1-WG3, symbol SystemDiagram:Cable12
- removed W33: RIO:ENC0-IMU:RIO ENC1, symbol SystemDiagram:Cable
- removed W34: RIO:ENC1-IMU:RIO ENC2, symbol SystemDiagram:Cable
- removed W35: RIO:DIO0-RIO:DIO1_IMU:RIO PWM, symbol SystemDiagram:Cable12
- removed W36: MOT6:CAN_W62, symbol SystemDiagram:Cable
- removed W37: DIO8-BBA2:OUT, symbol SystemDiagram:Cable
- removed W38: DIO9-BBA3:OUT, symbol SystemDiagram:Cable
- removed W39: VRM2:12V2A_ETH1:PWR, symbol SystemDiagram:Cable
- removed W4: MC1-W5-14AWG, symbol SystemDiagram:Cable
- removed W40: PI6_CAM3, symbol SystemDiagram:Cable
- removed W41: PI2_CAM2, symbol SystemDiagram:Cable
- removed W42: PI3_CAM1, symbol SystemDiagram:Cable
- removed W43: PI4_CAM4, symbol SystemDiagram:Cable
- removed W44: PI5_CAM5, symbol SystemDiagram:Cable
- removed W45: RADIO_RIO_ETH, symbol SystemDiagram:Cable
- removed W46: ETH1_PI2, symbol SystemDiagram:Cable
- removed W47: ETH1_PI3, symbol SystemDiagram:Cable
- removed W48: ETH1_PI4, symbol SystemDiagram:Cable
- removed W49: ETH1_PI5, symbol SystemDiagram:Cable
- removed W5: W4-MOT9-14AWG, symbol SystemDiagram:Cable
- removed W50: ETH1_PI6, symbol SystemDiagram:Cable
- removed W51: ETH1_PI1, symbol SystemDiagram:Cable
- removed W52: ETH1_RADIO, symbol SystemDiagram:Cable
- removed W53: VRM1_PWR, symbol SystemDiagram:Cable
- removed W55: IMU:ENC1-ENCA1, symbol SystemDiagram:WireTag
- removed W56: WG4-WG3_IND1_PWR, symbol SystemDiagram:Cable12
- removed W57: RIO:PWM0_FALCON-PROX:CAN, symbol SystemDiagram:Cable
- removed W58: RIO:PWM1_FALCON-DIST:CAN, symbol SystemDiagram:Cable
- removed W59: BBA2-W27, symbol SystemDiagram:Cable13
- removed W6: MC2-W7-14AWG, symbol SystemDiagram:Cable
- removed W60: BBA3-W27, symbol SystemDiagram:Cable13
- removed W61: RIO:CAN_IND1:CAN, symbol SystemDiagram:Cable
- removed W62: W36_MOT10:CAN, symbol SystemDiagram:Cable
- removed W63: WG10-WG11_PI6:PWR, symbol SystemDiagram:Cable12
- removed W64: W15-MGA3, symbol SystemDiagram:Cable
- removed W65: W16-MGA4, symbol SystemDiagram:Cable
- removed W66: WG8-WG9_PI6:PWR, symbol SystemDiagram:Cable12
- removed W67: PD:N-PI-PWR_WG6-WG7, symbol SystemDiagram:Cable12
- removed W68: WG6-WG7_PI2:PWR, symbol SystemDiagram:Cable12
- removed W69: WG6-WG7_PI3:PWR, symbol SystemDiagram:Cable12
- removed W7: W6-MOT11-14AWG, symbol SystemDiagram:Cable
- removed W70: PD:S-PI-PWR_WG10-WG11, symbol SystemDiagram:Cable12
- removed W71: WG10-WG11_PI5:PWR, symbol SystemDiagram:Cable12
- removed W72: RIO:CAN_PD1:CAN, symbol SystemDiagram:Cable
- removed W73: PD:DRV-PI-PWR_WG8-WG9, symbol SystemDiagram:Cable12
- removed W74: PD:IMU-PI-PWR_PI1, symbol SystemDiagram:Cable12
- removed W8: PD1:T4-W9-14AWG, symbol SystemDiagram:Cable
- removed W9: W8-MOT10-14AWG, symbol SystemDiagram:Cable
- removed WG1: 5V, symbol SystemDiagram:Wago_2
- removed WG10: 12V, symbol SystemDiagram:Wago_4
- removed WG11, WG7: GND, symbol SystemDiagram:Wago_4
- removed WG15: TOF_PWM, symbol SystemDiagram:Wago_2
- removed WG16: BB2, symbol SystemDiagram:Wago_2
- removed WG2: 12V, symbol SystemDiagram:Wago_5
- removed WG3: GND, symbol SystemDiagram:Wago_5
- removed WG4, WG8: 12V, symbol SystemDiagram:Wago_3
- removed WG5, WG9: GND, symbol SystemDiagram:Wago_3
- removed WG6: 12V_N_PI, symbol SystemDiagram:Wago_4
- added BB1: Intake BeamBreakSensor, symbol SystemDiagram:BeamBreakSensor
- added BB3: Amp Trap BeamBreakSensor, symbol SystemDiagram:BeamBreakSensor
- added BBA1: BeamBreakAdapter, symbol SystemDiagram:BeamBreakAdapter
- added MAG5: Climber Mag_Encoder, symbol SystemDiagram:Mag_Encoder
- added MOT11: Kraken Amp Trap, symbol SystemDiagram:Falcon_Motor
- added MOT12: Kraken Trap Extension, symbol SystemDiagram:Falcon_Motor
- added MOT13: Kraken Climber, symbol SystemDiagram:Falcon_Motor
- added MOT14: Kraken Deploy Intake, symbol SystemDiagram:Falcon_Motor
- added MOT9: Kraken Intake, symbol SystemDiagram:Falcon_Motor
- added POT5: Climber Pot, symbol SystemDiagram:Pot
- added W1: BT1:POS-CB1:1, symbol SystemDiagram:WireTag
- added W10: PD1:T14-MOT7:POWER, symbol SystemDiagram:WireTag
- added W11: PD1:T15-MOT8:POWER, symbol SystemDiagram:WireTag
- added W12: PD1:T4-MOT9:POWER, symbol SystemDiagram:WireTag
- added W13: PD1:T5-MOT14:POWER, symbol SystemDiagram:WireTag
- added W14: PD1:T6-MOT10:POWER, symbol SystemDiagram:WireTag
- added W15: PD1:T7-MOT12:POWER, symbol SystemDiagram:WireTag
- added W16: PD1:T8-MOT13:POWER, symbol SystemDiagram:WireTag
- added W2: BT1:NEG-PDB:VIN_NEG, symbol SystemDiagram:WireTag
- added W3: CB1:2-PD1:VIN_POS, symbol SystemDiagram:WireTag
- added W4: PD1:T0-MOT1:POWER, symbol SystemDiagram:WireTag
- added W5: PD1:T1-MOT2:POWER, symbol SystemDiagram:WireTag
- added W6: PD1:T12-MOT3:POWER, symbol SystemDiagram:WireTag
- added W7: PD1:T13-MOT4:POWER, symbol SystemDiagram:WireTag
- added W8: PD1:T2-MOT5:POWER, symbol SystemDiagram:WireTag
- added W9: PD1:T3-MOT6:POWER, symbol SystemDiagram:WireTag
- BB2: value CubeBeamBreakSensor -> Amp Trap BeamBreakSensor
- CB17: value 10A -> 30A
- ENC1: value SHAFT_ENC_DRV_R -> Left Shaft_Encoder
- ENC2: value SHAFT_ENC_DRV_L -> Right Shaft_Encoder
- MAG1: value MAG_ENC_PROX -> Shooter Elevation Mag_Encoder; MFG CTRE -> (none); MFG P/N SRX MAG ENCODER -> (none)
- MAG2: value MAG_ENC_DIST -> Shooter Yaw Mag_Encoder; MFG CTRE -> (none); MFG P/N SRX MAG ENCODER -> (none)
- MAG3: value MAG_ENC_ROLL -> Deploy Intake Mag_Encoder; MFG CTRE -> (none); MFG P/N SRX MAG ENCODER -> (none)
- MAG4: value MAG_ENC_WRIST -> Trap Extension Mag_Encoder; MFG CTRE -> (none); MFG P/N SRX MAG ENCODER -> (none)
- MOT1: value FALCON_DRV_RIGHT_FRONT -> Kraken Left Front Drive Motor
- MOT10: value FALCON_INTAKE -> Kraken Transfer
- MOT2: value FALCON_DRV_RIGHT_BACK -> Kraken Left Back Drive Motor
- MOT3: value FALCON_DRV_RIGHT_UNDER -> Kraken Right Front Drive Motor
- MOT4: value FALCON_DRV_LEFT_FRONT -> Kraken Right Back Drive Motor
- MOT5: value FALCON_DRV_LEFT_BACK -> Kraken Shooter 1
- MOT6: value FALCON_DRV_LEFT_UNDER -> Kraken Shooter 2
- MOT7: value FALCON_PROX -> Kraken Shooter Elevation
- MOT8: value FALCON_DIST -> Kraken Shooter Yaw
- POT1: value POT_PROX -> Shooter Elevation Pot
- POT2: value POT_DIST -> Shooter Yaw Pot
- POT3: value POT_ROLL -> Deploy Intake Pot
- POT4: value POT_WRIST -> Trap Extension Pot
Connections:
- net N_PI_PWR is gone; now on net NX POWER: PD1.T11
- net WRIST_PWR is gone; now on net TRANSFER: PD1.T6
- net LEFT_BACK_DRIVE_PWR: now also W5.
- net LEFT_FRONT_DRIVE_PWR: now also W4.
- net RIGHT_BACK_DRIVE_PWR: now also MOT4. (PWR), PD1.T13, W7.; no longer MOT5. (PWR), PD1.T14
- net RIGHT_FRONT_DRIVE_PWR: now also MOT3. (PWR), PD1.T12, W6.; no longer MOT4. (PWR), PD1.T13
- net at VRM1. (5V/2A): now also W54.1
- net at POE?. (RJ45S): now also RDO1. (POWER); no longer VRM1. (5V/2A)
- net at W54.1: now also RDO1. (POWER); no longer VRM1. (5V/2A)
- net at RIO1.CAN: now also PD1.CAN
- net at RIO1.INPUT_V (P_IN): now also PD1.CTLR_PWR
- net at RIO1.USB2: no longer CAN1. (USB)
- net at MGA1. (POT): now also POT2. (OUT)
- net TRANSFER: now reaches MOT10. (PWR)
- net TRANSFER: now also W14.
- net at MGA2. (POT): now also MAG3. (OUT)
- net at MAG2. (OUT): now also MGA1. (POT)
- net SHOOTER YAW: now reaches MOT8. (PWR)
- net SHOOTER YAW: now also PD1.T15, W11.
- net at CB1.CB: now also BT1.1 (+), W1.
- net at MGA4. (POT): now also POT4. (OUT)
- net at BBA3. (SNSR): now also BB1. (OUT)
- net SHOOTER2: now reaches MOT6. (PWR)
- net SHOOTER2: now also PD1.T3, W9.
- net SHOOTER1: now reaches MOT5. (PWR)
- net SHOOTER1: now also PD1.T2, W8.; no longer MOT6. (PWR)
- net NX POWER: now reaches PD2. (IN)
- net at MAG4. (OUT): now also MGA4. (POT)
- net at POT3. (OUT): now also MGA2. (POT)
- net at BT1.2 (-): now also PD1.VIN_NEG, W2.
- net SHOOTER ELEVATION: now reaches MOT7. (PWR)
- net SHOOTER ELEVATION: now also PD1.T14, W10.
- net at PD1.VIN_POS: now also CB1.CB, W3.
- net CAN_FD: no longer names the net of CAN1. (USB)
- net CAN_FD: no longer MOT1. (PWR)
- net CONE_POSITION_PWM: no longer names the net of RIO1.DIO8
- net CUBE_BEAM_BREAK: no longer names the net of RIO1.DIO7
- net DISTAL_POT_MAG_ENCODER: no longer names the net of RIO1.ENC_AD2
- net DISTAL_PWM: no longer names the net of RIO1.PWM0
- removed net DISTAL_PWR: MOT8. (PWR), PD1.T12
- net DRIVE_ENC_LEFT: no longer names the net of RIO1.ENC1
- net DRIVE_ENC_RIGHT: no longer names the net of RIO1.ENC0
- net DRV_PI_PWR: no longer names the net of PD1.T9
- net HEADING_PWM: no longer names the net of RIO1.DIO1
- net IMU_PI_PWR renamed CLIMBER
- net CLIMBER: now also MOT13. (PWR), W16.
- net INTAKE_PWR renamed INTAKE
- net INTAKE: now also MOT9. (PWR), W12.
- net PROXIMAL_POT_MAG_ENCODER: no longer names the net of RIO1.ENC_AD3
- net PROXIMAL_PWM: no longer names the net of RIO1.PWM1
- removed net PROXIMAL_PWR: MOT7. (PWR), PD1.T3
- net PSU_PWR renamed TRAP EXTENSION
- net TRAP EXTENSION: now also MOT12. (PWR), W15.
- net ROLL_POT_MAG_ENCODER: no longer names the net of RIO1.ENC_AD5
- net ROLL_PWM: no longer names the net of RIO1.PWM3
- net ROLL_PWR renamed DEPLOY INTAKE
- net DEPLOY INTAKE: now also MOT14. (PWR), W13.
- net S_PI_PWR: no longer names the net of PD1.T10
- net WRIST_POT_MAG_ENCODER: no longer names the net of RIO1.ENC_AD4
- net WRIST_PWM: no longer names the net of RIO1.PWM2
- net YAW_RATE_PWM: no longer names the net of RIO1.DIO0
- new net: POE?. (RJ45S), VRM1. (5V/2A)
- new net: MAG5. (OUT), MGA3. (POT)
- new net: BB3. (OUT), BBA1. (SNSR)
- new net: MGA3. (POT), POT5. (OUT)
- now unconnected: BBA2. (SNSR), BBA2. (SNSR), MGA3. (POT), MGA3. (POT)
- no-connect marks 15 -> 0
Other:
- note removed: "ARM"
- note removed: "CAN_ID=1"
- note removed: "CAN_ID=2"
- note removed: "CAN_ID=3"
- note removed: "CAN_ID=4"
- note removed: "CAN_ID=5"
- note removed: "CAN_ID=6"
- note removed: "DISTAL"
- note removed: "INTAKE"
- note removed: "LEFT DRIVE"
- note removed: "PROXIMAL"
- note removed: "RIGHT DRIVE"
- note removed: "ROLL"
- note removed: "WRIST"
- moved on the sheet: CAN1, F1, F2, F3, F4, F5, PD2, POE?, RDO1, RIO1, VRM1, W54
