File: robots/2024/system-drawing/kicad-schematic/2024-SystemDiagram.kicad_sch (KiCad schematic)
At the start: 87 parts

Commit message: System diagram update.  Initial wiring complete
Signed-off-by: Scott Berman <sgberman1@gmail.com>
Parts:
- removed W54: VRM1:12V2A_RDO1:PWR, symbol SystemDiagram:Cable
- added CAM1, CAM2, CAM3, CAM4: Camera, symbol SystemDiagram:Camera
- added CAN2, CAN3, CAN4, CAN5: CAN_Terminator, symbol SystemDiagram:CAN_Terminator
- added ETH1: Ethernet_Switch, symbol SystemDiagram:Ethernet_Switch
- added IMU1: IMU2x, symbol SystemDiagram:IMU2x
- added IND1: CANdle, symbol SystemDiagram:CANdle
- added MAG6: Catapult Mag_Encoder, symbol SystemDiagram:Mag_Encoder
- added MGA5, MGA6: MagEncoderAdapter, symbol SystemDiagram:MagEncoderAdapter
- added MOT15: Kraken Note Retention, symbol SystemDiagram:Falcon_Motor
- added POT6: Catapult Pot, symbol SystemDiagram:Pot
- added RSL1: RSL, symbol SystemDiagram:RSL
- added VRM2: VRM, symbol SystemDiagram:VRM
- added W17: DUMP ROLLERS PWR, symbol SystemDiagram:WireTag
- added W18: NOTE RETENTION PWR, symbol SystemDiagram:WireTag
- added W19: PDF PWR, symbol SystemDiagram:WireTag
- added W20: Catapult Mag Encoder, symbol SystemDiagram:WireTag
- added W21: Catapult Pot, symbol SystemDiagram:WireTag
- added W22: Left Shaft Encoder, symbol SystemDiagram:WireTag
- added W23: Right Shaft Encoder, symbol SystemDiagram:WireTag
- added W24: Catapult Beam Break, symbol SystemDiagram:WireTag
- added W25: Cat Altitude Mag Encoder, symbol SystemDiagram:WireTag
- added W26: Cat Altitude Pot, symbol SystemDiagram:WireTag
- added W27: Cat Turret Mag Encoder, symbol SystemDiagram:WireTag
- added W28: Cat Turret Pot, symbol SystemDiagram:WireTag
- added W29: Intake Pivot Pot, symbol SystemDiagram:WireTag
- added W30: Intake Mag Encoder, symbol SystemDiagram:WireTag
- added W31: Climber Mag Encoder, symbol SystemDiagram:WireTag
- added W32: Trap Extend Mag Encoder, symbol SystemDiagram:WireTag
- added W33: Trap Extend Pot, symbol SystemDiagram:WireTag
- added W34: Climber Pot, symbol SystemDiagram:WireTag
- added W35: Transfer Roller Beam Break, symbol SystemDiagram:WireTag
- added W36: Dump Beam Break, symbol SystemDiagram:WireTag
- added W37: USBA-B, symbol SystemDiagram:WireTag
- added W38: NX1 PWR, symbol SystemDiagram:WireTag
- added W39: NX2 PWR, symbol SystemDiagram:WireTag
- added W40: IMU NX PWR, symbol SystemDiagram:WireTag
- added W41: IMU PWR, symbol SystemDiagram:WireTag
- added W42: NX1 CAMERA A, symbol SystemDiagram:WireTag
- added W43: NX1 CAMERA B, symbol SystemDiagram:WireTag
- added W44: NX2 CAMERA A, symbol SystemDiagram:WireTag
- added W45: NX2 CAMERA B, symbol SystemDiagram:WireTag
- added W46, W47, W48: IMU CAN, symbol SystemDiagram:WireTag
- added W49: CTLR PWR, symbol SystemDiagram:WireTag
- added W50: CATAPULT1 PWM, symbol SystemDiagram:WireTag
- added W51: CATAPULT2 PWM, symbol SystemDiagram:WireTag
- added W52: CANdle PWR, symbol SystemDiagram:WireTag
- added W53: CAT ENC POT RIO, symbol SystemDiagram:WireTag
- added W54: CAT BEAM BREAK RIO, symbol SystemDiagram:WireTag
- added W55: CAT ALTITUDE ENC POT RIO, symbol SystemDiagram:WireTag
- added W56: CAT TURRET ENC POT RIO, symbol SystemDiagram:WireTag
- added W57: INTAKE PIVOT ENC POT RIO, symbol SystemDiagram:WireTag
- added W58: TRANSFER ROLLER BEAM BREAK RIO, symbol SystemDiagram:WireTag
- added W59: TRAP EXTEND ENC POT RIO, symbol SystemDiagram:WireTag
- added W60: CLIMBER ENC POT RIO, symbol SystemDiagram:WireTag
- added W61: DUMP BEAM BREAK RIO, symbol SystemDiagram:WireTag
- added W62: RSL, symbol SystemDiagram:WireTag
- added W63: CAT BB PWR, symbol SystemDiagram:WireTag
- added W64: TRANSFER ROLLER BB PWR, symbol SystemDiagram:WireTag
- added W65: DUMP BB PWR, symbol SystemDiagram:WireTag
- added W66: VRM1 PWR, symbol SystemDiagram:WireTag
- added W67: CANivore PWR, symbol SystemDiagram:WireTag
- added W68, W69, W70, W71, W72, W73, W74, W75, W76, W77, W78, W79, W80, W81, W82, W83: CAN, symbol SystemDiagram:WireTag
- added W84: ETH SW PWR, symbol SystemDiagram:WireTag
- added W85: VRM2 PWR, symbol SystemDiagram:WireTag
- added W86: ETH RIO, symbol SystemDiagram:WireTag
- added W87: ETH NX1, symbol SystemDiagram:WireTag
- added W88: ETH NX2, symbol SystemDiagram:WireTag
- added W89: ETH IMU NX, symbol SystemDiagram:WireTag
- added W90: IMU HEADING, symbol SystemDiagram:WireTag
- added WG1: Wago_4, symbol SystemDiagram:Wago_4
- A1: value Orin NX1 -> NX1
- A2: value Orin NX2 -> NX2
- A3: value Orin NX3 -> IMU NX
- BB1: value Intake BeamBreakSensor -> Dump BeamBreakSensor; MFG (none) -> Automation Direct; MFG P/N (none) -> QMI7-0N-0F
- BB2: value Amp Trap BeamBreakSensor -> Catapult BeamBreakSensor; MFG (none) -> Automation Direct; MFG P/N (none) -> QMI7-0N-0F
- BB3: value Amp Trap BeamBreakSensor -> Tranfer Roller BeamBreakSensor; MFG (none) -> Automation Direct; MFG P/N (none) -> QMI7-0N-0F
- MAG1: value Shooter Elevation Mag_Encoder -> Catapult Altitude Mag_Encoder
- MAG2: value Shooter Yaw Mag_Encoder -> Catapult Turret Mag_Encoder
- MAG3: value Deploy Intake Mag_Encoder -> Intake Pivot Mag_Encoder
- MAG4: value Trap Extension Mag_Encoder -> Trap Extend Mag_Encoder
- MOT10: value Kraken Transfer -> Kraken Transfer Rollers
- MOT11: value Kraken Amp Trap -> Kraken Dump Rollers
- MOT12: value Kraken Trap Extension -> Kraken Extend
- MOT14: value Kraken Deploy Intake -> Kraken Intake Pivot
- MOT5: value Kraken Shooter 1 -> Kraken Catapult 1
- MOT6: value Kraken Shooter 2 -> Kraken Catapult 2
- MOT7: value Kraken Shooter Elevation -> Kraken Catapult Altitude
- MOT8: value Kraken Shooter Yaw -> Kraken Catapult Turret
- MOT9: value Kraken Intake -> Kraken Intake Roller
- POT1: value Shooter Elevation Pot -> Catapult Altitude Pot
- POT2: value Shooter Yaw Pot -> Catapult Turret Pot
- POT3: value Deploy Intake Pot -> Intake Pivot Pot
- POT4: value Trap Extension Pot -> Trap Extend Pot
- W10: value PD1:T14-MOT7:POWER -> CATAPULT ALTITUDE PWR
- W11: value PD1:T15-MOT8:POWER -> CATAPULT TURRET PWR
- W12: value PD1:T4-MOT9:POWER -> INTAKE ROLLER PWR
- W13: value PD1:T5-MOT14:POWER -> INTAKE PIVOT PWR
- W14: value PD1:T6-MOT10:POWER -> TRANSFER ROLLER PWR
- W15: value PD1:T7-MOT12:POWER -> EXTEND PWR
- W16: value PD1:T8-MOT13:POWER -> CLIMBER PWR
- W4: value PD1:T0-MOT1:POWER -> LEFT FRONT DRIVE PWR
- W5: value PD1:T1-MOT2:POWER -> LEFT BACK DRIVE PWR
- W6: value PD1:T12-MOT3:POWER -> RIGHT FRONT DRIVE PWR
- W7: value PD1:T13-MOT4:POWER -> RIGHT BACK DRIVE PWR
- W8: value PD1:T2-MOT5:POWER -> CATAPULT1 PWR
- W9: value PD1:T3-MOT6:POWER -> CATAPULT2 PWR
Connections:
- net CLIMBER is gone; now on net CLIMBER PWR: MOT13. (PWR), PD1.T8, W16.
- net DEPLOY INTAKE is gone; now on net INTAKE PIVOT PWR: MOT14. (PWR), PD1.T5, W13.
- net INTAKE is gone; now on net INTAKE ROLLER PWR: MOT9. (PWR), PD1.T4, W12.
- net LEFT_BACK_DRIVE_PWR is gone; now on net LEFT BACK DRIVE PWR: MOT2. (PWR), PD1.T1, W5.
- net LEFT_FRONT_DRIVE_PWR is gone; now on net LEFT FRONT DRIVE PWR: MOT1. (PWR), PD1.T0, W4.
- net NX POWER is gone; now on net PDF POWER: PD1.T11, PD2. (IN)
- net RIGHT_BACK_DRIVE_PWR is gone; now on net RIGHT BACK DRIVE PWR: MOT4. (PWR), PD1.T13, W7.
- net RIGHT_FRONT_DRIVE_PWR is gone; now on net RIGHT FRONT DRIVE PWR: MOT3. (PWR), PD1.T12, W6.
- net SHOOTER ELEVATION is gone; now on net CATAPULT ALTITUDE PWR: MOT7. (PWR), PD1.T14, W10.
- net SHOOTER YAW is gone; now on net CATAPULT TURRET PWR: MOT8. (PWR), PD1.T15, W11.
- net SHOOTER1 is gone; now on net CATAPULT1 PWR: MOT5. (PWR), PD1.T2, W8.
- net SHOOTER2 is gone; now on net CATAPULT2 PWR: MOT6. (PWR), PD1.T3, W9.
- net TRANSFER is gone; now on net TRANSFER ROLLER PWR: MOT10. (PWR), PD1.T6, W14.
- net TRAP EXTENSION is gone; now on net EXTEND PWR: MOT12. (PWR), PD1.T7, W15.
- net CAN_PD: now also MOT7. (PWR), W82.
- net VRM1_PWR: now also VRM1. (5V/2A), W66.
- net VRM2_PWR: now also VRM2. (5V/2A), W85.
- net at POE?. (RJ45S): now also RDO1. (POWER); no longer VRM1. (5V/2A)
- net CATAPULT TURRET PWR: now reaches MOT8. (PWR)
- net at PD1.CAN, RIO1.CAN: now also W83.
- net CAT BEAM BREAK: now reaches RIO1.DIO22
- net CAT BEAM BREAK: now also BBA2. (SNSR), W54.
- net TRANSFER ROLLER BEAM BREAK: now reaches RIO1.DIO23
- net TRANSFER ROLLER BEAM BREAK: now also BBA1. (SNSR), W58.
- net DUMP BEAM BREAK: now reaches RIO1.DIO24
- net DUMP BEAM BREAK: now also BBA3. (SNSR), W61.
- net IMU HEADING: now reaches RIO1.DIO25
- net IMU HEADING: now also IMU1. (RIO_PWM2), W90.
- net LEFT ENC: now reaches RIO1.DIO6
- net LEFT ENC: now also ENC1. (OUT), RIO1.DIO7, W22.
- net RIGHT ENC: now reaches RIO1.DIO8
- net RIGHT ENC: now also ENC2. (OUT), RIO1.DIO9, W23.
- net CAT ENC POT RIO: now reaches RIO1.ENC_AD0
- net CAT ENC POT RIO: now also MGA4. (POT), RIO1.ENC_AD4, MGA5. (POT), W53., W59.
- net CAT ALTITUDE ENC POT RIO: now reaches RIO1.ENC_AD1
- net CAT ALTITUDE ENC POT RIO: now also MGA6. (POT), W55.
- net CAT TURRET ENC POT RIO: now reaches RIO1.ENC_AD2
- net CAT TURRET ENC POT RIO: now also MGA1. (POT), W56.
- net at RIO1.ENC_AD3: now also MGA2. (POT), W57.
- net CLIMBER ENC POT RIO: now reaches RIO1.ENC_AD5
- net CLIMBER ENC POT RIO: now also MGA3. (POT), W60.
- net at RIO1.ETH: now also ETH1. (POWER), W86.
- net at PD1.CTLR_PWR, RIO1.INPUT_V (P_IN): now also W49.
- net CATAPULT1 PWM: now reaches RIO1.PWM0
- net CATAPULT1 PWM: now also MOT5. (PWR), W50.
- net CATAPULT2 PWM: now reaches RIO1.PWM1
- net CATAPULT2 PWM: now also MOT6. (PWR), W51.
- net at RIO1.RSL: now also RSL1. (P), W62.
- net at RIO1.USB2: now also CAN1. (USB), W37.
- net NX2 PWR: now reaches A2. (Power)
- net NX2 PWR: now also PD2. (IN), W39.
- net at RDO1. (POWER): now also ETH1. (POWER); no longer POE?. (RJ45S)
- net at MAG4. (OUT), MGA4. (POT): now also W32.
- net at MGA2. (POT): now also MAG3. (OUT), W30.
- net at MGA2. (POT), POT3. (OUT): now also W29.
- net at MGA4. (POT), POT4. (OUT): now also W33.
- net EXTEND PWR: now reaches MOT12. (PWR)
- net at MAG2. (OUT), MGA1. (POT): now also W27.
- net TRANSFER ROLLER PWR: now reaches MOT10. (PWR)
- net at MAG1. (OUT): now also MGA6. (POT), W25.
- net at MAG5. (OUT), MGA3. (POT): now also W31.
- net LEFT BACK DRIVE PWR: now reaches MOT2. (PWR)
- net at BB2. (OUT): now also BBA2. (SNSR), W24.
- net LEFT FRONT DRIVE PWR: now reaches MOT1. (PWR)
- net CATAPULT2 PWR: now reaches MOT6. (PWR)
- net at POT1. (OUT): now also MGA6. (POT), W26.
- net PDF POWER: now reaches PD2. (IN)
- net PDF POWER: now also W19.
- net at BB1. (OUT), BBA3. (SNSR): now also W36.
- net INTAKE ROLLER PWR: now reaches MOT9. (PWR)
- net IMU NX PWR: now reaches A3. (Power)
- net IMU NX PWR: now also PD2. (IN), W40.
- net CATAPULT ALTITUDE PWR: now reaches MOT7. (PWR)
- net at MGA1. (POT), POT2. (OUT): now also W28.
- net NX1 PWR: now reaches A1. (Power)
- net NX1 PWR: now also PD2. (IN), W38.
- net at BB3. (OUT), BBA1. (SNSR): now also W35.
- net CLIMBER PWR: now reaches MOT13. (PWR)
- net DUMP ROLLERS PWR: now reaches MOT11. (PWR)
- net DUMP ROLLERS PWR: now also PD1.T9, W17.
- net at MGA3. (POT), POT5. (OUT): now also W34.
- net INTAKE PIVOT PWR: now reaches MOT14. (PWR)
- net RIGHT BACK DRIVE PWR: now reaches MOT4. (PWR)
- net NOTE RETENTION PWR: now reaches PD1.T10
- net NOTE RETENTION PWR: now also MOT15. (PWR), W18.
- net RIGHT FRONT DRIVE PWR: now reaches MOT3. (PWR)
- net CAN_FD_CANivore: now reaches CAN1. (USB)
- net CAN_FD_CANivore: now also MOT1. (PWR)
- net CATAPULT1 PWR: now reaches MOT5. (PWR)
- new net: VRM1. (5V/2A), WG1. (4)
- new net: POE?. (RJ45S), VRM1. (5V/2A)
- new net: RDO1. (POWER), VRM1. (5V/2A)
- new net: CAN1. (USB), W67., WG1. (4)
- new net: MOT7. (PWR), MOT8. (PWR), W71.
- new net: MOT8. (PWR), MOT9. (PWR), W72.
- new net: MOT11. (PWR), MOT13. (PWR), W77.
- new net: MOT11. (PWR), MOT15. (PWR), W78.
- new net: MOT14. (PWR), MOT9. (PWR), W73.
- new net: A2. (Power), ETH1. (POWER), W88.
- new net: A2. (Power), CAM3., W44.
- new net: A2. (Power), CAM4., W45.
- new net: IND1. (P), MOT15. (PWR), W79.
- new net: MOT10. (PWR), MOT12. (PWR), W75.
- new net: MOT12. (PWR), MOT13. (PWR), W76.
- new net: CAN5., IND1. (P), W80.
- new net: MOT10. (PWR), MOT14. (PWR), W74.
- new net: ETH1. (POWER), VRM2. (5V/2A), W84.
- new net: A3. (Power), ETH1. (POWER), W89.
- new net: A1. (Power), ETH1. (POWER), W87.
- new net: MOT1. (PWR), MOT2. (PWR), W68.
- new net: MOT2. (PWR), MOT3. (PWR), W69.
- new net: A3. (Power), CAN2., W46.
- new net: CAN4., MOT4. (PWR), W81.
- new net: MOT3. (PWR), MOT4. (PWR), W70.
- new net: A3. (Power), IMU1. (RIO_PWM2), W47.
- new net: A1. (Power), CAM2., W43.
- new net: CAN3., IMU1. (RIO_PWM2), W48.
- new net: MAG6. (OUT), MGA5. (POT), W20.
- new net: MGA5. (POT), POT6. (OUT), W21.
- new net: A1. (Power), CAM1., W42.
- new net CANdle PWR: IND1. (P), PD2. (IN), W52.
- new net CAT BB PWR: BBA2. (SNSR), W63., WG1. (4)
- new net DUMP BB PWR: BBA3. (SNSR), VRM1. (5V/2A), W65.
- new net IMU PWR: IMU1. (RIO_PWM2), PD2. (IN), W41.
- new net TRANSFER ROLLER BB PWR: BBA1. (SNSR), W64., WG1. (4)
- no-connect marks 0 -> 46
Other:
- note added: "A"
- note added: "B"
- note added: "INTAKE PIVOT ENC POT RIO"
- moved on the sheet: A1, A2, A3, BB1, BB3, BBA1, BBA3, F1, F2, F3, F4, F5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

Commit message: Fixed system drawing
Signed-off-by: Scott Berman <sgberman1@gmail.com>
Parts:
- CB14, CB15, CB16: value 10A -> 30A
- gave numbers to parts that had none: 1
- renumbered LINK to LINK1
Connections:
- net CAT ENC POT RIO: no longer MGA4. (POT), RIO1.ENC_AD4, W59.
- net at POE1. (RJ45S): now also RDO1. (POWER); no longer VRM1. (5V/2A)
- net at RDO1. (POWER): now also ETH1. (POWER); no longer VRM1. (5V/2A)
- net INTAKE PIVOT ENC POT RIO: now reaches MGA2. (POT), RIO1.ENC_AD3, W57.
- net at ETH1. (POWER): now also A1. (Power), W87.; no longer RDO1. (POWER)
- new net: VRM1. (5V/2A), WG1. (4)
- new net: POE1. (RJ45S), VRM1. (5V/2A)
- new net: RDO1. (POWER), VRM1. (5V/2A)
- new net: CAN1. (USB), W67., WG1. (4)
- new net: MOT7. (PWR), MOT8. (PWR), W71.
- new net: MOT8. (PWR), MOT9. (PWR), W72.
- new net: MOT11. (PWR), MOT13. (PWR), W77.
- new net: MOT11. (PWR), MOT15. (PWR), W78.
- new net: MOT14. (PWR), MOT9. (PWR), W73.
- new net: A2. (Power), ETH1. (POWER), W88.
- new net: IND1. (P), MOT15. (PWR), W79.
- new net: MOT10. (PWR), MOT12. (PWR), W75.
- new net: MOT12. (PWR), MOT13. (PWR), W76.
- new net: MOT10. (PWR), MOT14. (PWR), W74.
- new net: ETH1. (POWER), VRM2. (5V/2A), W84.
- new net: A3. (Power), ETH1. (POWER), W89.
- new net: MOT1. (PWR), MOT2. (PWR), W68.
- new net: MOT2. (PWR), MOT3. (PWR), W69.
- new net: MOT3. (PWR), MOT4. (PWR), W70.
- new net: A3. (Power), IMU1. (RIO_PWM2), W47.
- new net TRAP EXTEND ENC POT RIO: MGA4. (POT), RIO1.ENC_AD4, W59.
Other:
- note removed: "INTAKE PIVOT ENC POT RIO"
- moved on the sheet: BBA1
Changed lines of the file:
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@@
   (junction (at 173.99 205.74) (diameter 0) (color 0 0 0 0)
   )
-  (junction (at 260.35 182.88) (diameter 0) (color 0 0 0 0)
-  )
   (junction (at 487.68 368.3) (diameter 0) (color 0 0 0 0)
   )
@@
   (junction (at 240.03 424.18) (diameter 0) (color 0 0 0 0)
   )
-  (junction (at 260.35 184.15) (diameter 0) (color 0 0 0 0)
-  )
   (junction (at 170.18 283.21) (diameter 0) (color 0 0 0 0)
   )
@@
     (stroke (width 0.508) (type default) (color 255 0 0 1))
   )
-  (wire (pts (xy 260.35 194.31) (xy 260.35 184.15))
-    (stroke (width 0.254) (type default) (color 194 0 194 1))
-  )
   (wire (pts (xy 304.8 242.57) (xy 220.98 242.57))
     (stroke (width 0.254) (type default) (color 194 0 194 1))
@@
     (stroke (width 0.508) (type default) (color 255 0 0 1))
   )
-  (wire (pts (xy 543.56 339.09) (xy 553.72 339.09))
+  (wire (pts (xy 543.56 339.09) (xy 552.45 339.09))
     (stroke (width 0.254) (type default) (color 255 0 0 1))
   )
@@
     (stroke (width 0.508) (type default) (color 255 0 0 1))
   )
-  (wire (pts (xy 401.32 182.88) (xy 260.35 182.88))
-    (stroke (width 0.254) (type default) (color 194 0 194 1))
-  )
   (wire (pts (xy 231.14 388.62) (xy 240.03 388.62))
     (stroke (width 0.254) (type default) (color 0 194 194 1))
@@
     (stroke (width 0.508) (type default) (color 255 0 0 1))
   )
-  (wire (pts (xy 576.58 340.36) (xy 586.74 340.36))
+  (wire (pts (xy 575.31 340.36) (xy 586.74 340.36))
     (stroke (width 0) (type default))
   )
@@
     (stroke (width 0) (type default))
   )
-  (wire (pts (xy 401.32 182.88) (xy 401.32 368.3))
-    (stroke (width 0.254) (type default) (color 194 0 194 1))
-  )
   (wire (pts (xy 270.51 207.01) (xy 487.68 207.01))
     (stroke (width 0.254) (type default) (color 194 0 194 1))
@@
     (stroke (width 0.508) (type default) (color 255 0 0 1))
   )
-  (wire (pts (xy 487.68 341.63) (xy 553.72 341.63))
+  (wire (pts (xy 487.68 341.63) (xy 552.45 341.63))
     (stroke (width 0.254) (type default) (color 194 0 194 1))
   )
@@
     (stroke (width 0.254) (type default) (color 255 0 0 1))
   )
-  (wire (pts (xy 260.35 158.75) (xy 260.35 182.88))
+  (wire (pts (xy 260.35 158.75) (xy 260.35 184.15))
     (stroke (width 0.254) (type default) (color 194 0 194 1))
   )
@@
     (stroke (width 0.254) (type default) (color 255 153 0 1))
   )
-  (wire (pts (xy 220.98 194.31) (xy 260.35 194.31))
+  (wire (pts (xy 220.98 194.31) (xy 401.32 194.31))
     (stroke (width 0.254) (type default) (color 194 0 194 1))
   )
@@
     (stroke (width 0.254) (type default) (color 0 194 194 1))
   )
+  (wire (pts (xy 401.32 194.31) (xy 401.32 368.3))
+    (stroke (width 0.254) (type default) (color 194 0 194 1))
+  )
   (wire (pts (xy 91.44 251.46) (xy 91.44 256.54))
     (stroke (width 0.254) (type default) (color 255 0 0 1))
@@
     (stroke (width 0.508) (type default) (color 255 0 0 1))
   )
-  (wire (pts (xy 260.35 182.88) (xy 260.35 184.15))
-    (stroke (width 0.254) (type default) (color 194 0 194 1))
-  )
   (wire (pts (xy 237.49 237.49) (xy 220.98 237.49))
     (stroke (width 0.254) (type default) (color 194 0 194 1))
@@
     (effects (font (size 1.27 1.27)) (justify left bottom))
   )
-  (text "INTAKE PIVOT ENC POT RIO" (at 222.25 191.77 0)
-    (effects (font (size 1.27 1.27)) (justify left bottom))
-  )
   (text "B" (at 222.25 240.03 0)
     (effects (font (size 1.27 1.27)) (justify left bottom))
@@
     (effects (font (size 1.27 1.27)) (justify left bottom))
   )
+  (label "INTAKE PIVOT ENC POT RIO" (at 222.25 191.77 0) (fields_autoplaced)
+    (effects (font (size 1.27 1.27)) (justify left bottom))
+  )
   (label "VRM2_PWR" (at 43.18 269.24 180) (fields_autoplaced)
     (effects (font (size 1.27 1.27)) (justify right bottom))
@@
   (symbol (lib_id "SystemDiagram:POE_Injector") (at 222.25 330.2 180) (unit 1)
     (in_bom yes) (on_board yes) (dnp no)
-    (property "Reference" "POE?" (at 217.17 331.47 0)
+    (property "Reference" "POE1" (at 217.17 331.47 0)
       (effects (font (size 1.27 1.27)) (justify left))
     )
@@
       (project "2024-SystemDiagram"
         (path "/12a52703-e3f4-4774-b510-3055ab1abf35"
-          (reference "POE?") (unit 1)
+          (reference "POE1") (unit 1)
         )
       )
@@
       (effects (font (size 1.27 1.27)))
     )
-    (property "Value" "10A" (at 213.36 119.38 0)
+    (property "Value" "30A" (at 213.36 119.38 0)
       (effects (font (size 1.27 1.27)))
     )
@@
       (effects (font (size 1.27 1.27)))
     )
-    (property "Value" "10A" (at 213.36 123.19 0)
+    (property "Value" "30A" (at 213.36 123.19 0)
       (effects (font (size 1.27 1.27)))
     )
@@
       (effects (font (size 1.27 1.27)))
     )
-    (property "Value" "10A" (at 213.36 127 0)
+    (property "Value" "30A" (at 213.36 127 0)
       (effects (font (size 1.27 1.27)))
     )
@@
   (symbol (lib_id "Graphic:SYM_Arrow_Large") (at 749.3 508 0) (unit 1)
     (in_bom no) (on_board no) (dnp no)
-    (property "Reference" "LINK" (at 749.3 505.714 0)
+    (property "Reference" "LINK1" (at 749.3 505.714 0)
       (effects (font (size 1.27 1.27)) hide)
     )
@@
       (project "2024-SystemDiagram"
         (path "/12a52703-e3f4-4774-b510-3055ab1abf35"
-          (reference "LINK") (unit 1)
+          (reference "LINK1") (unit 1)
         )
       )
@@
     )
   )
-  (symbol (lib_id "SystemDiagram:BeamBreakAdapter") (at 558.8 336.55 0) (unit 1)
+  (symbol (lib_id "SystemDiagram:BeamBreakAdapter") (at 557.53 336.55 0) (unit 1)
     (in_bom yes) (on_board yes) (dnp no)
-    (property "Reference" "BBA1" (at 565.15 331.47 0)
+    (property "Reference" "BBA1" (at 563.88 331.47 0)
       (effects (font (size 1.27 1.27)))
     )
-    (property "Value" "BeamBreakAdapter" (at 567.69 334.01 0)
+    (property "Value" "BeamBreakAdapter" (at 566.42 334.01 0)
       (effects (font (size 1.27 1.27)))
     )
-    (property "Footprint" "" (at 558.8 336.55 0)
+    (property "Footprint" "" (at 557.53 336.55 0)
       (effects (font (size 1.27 1.27)) hide)
     )
-    (property "Datasheet" "Components/beambreak-sch-20Jan2024.pdf" (at 558.8 336.55 0)
+    (property "Datasheet" "Components/beambreak-sch-20Jan2024.pdf" (at 557.53 336.55 0)
       (effects (font (size 1.27 1.27)) hide)
     )

Commit message: Changed CAN ref des to number greater than 100 to allow future change
Signed-off-by: Scott Berman <sgberman1@gmail.com>
Parts:
- added W103: CAN, symbol SystemDiagram:WireTag
- renumbered W82 to W101, W83 to W102, W81 to W104, W68 to W105, W69 to W106, W70 to W107, W71 to W108, W72 to W109, W73 to W110, W74 to W111, W75 to W112, W76 to W113, W77 to W114, W78 to W115, W79 to W116, W80 to W117
Connections:
- net CAN_FD_CANivore: now also W103.
- net at POE1. (RJ45S): now also RDO1. (POWER); no longer VRM1. (5V/2A)
- net at RDO1. (POWER): now also ETH1. (POWER); no longer VRM1. (5V/2A)
- net at ETH1. (POWER): now also A1. (Power), W87.; no longer RDO1. (POWER)
- new net: VRM1. (5V/2A), WG1. (4)
- new net: POE1. (RJ45S), VRM1. (5V/2A)
- new net: RDO1. (POWER), VRM1. (5V/2A)
- new net: CAN1. (USB), W67., WG1. (4)
- new net: MOT7. (PWR), MOT8. (PWR), W108.
- new net: MOT8. (PWR), MOT9. (PWR), W109.
- new net: MOT11. (PWR), MOT13. (PWR), W114.
- new net: MOT11. (PWR), MOT15. (PWR), W115.
- new net: MOT14. (PWR), MOT9. (PWR), W110.
- new net: A2. (Power), ETH1. (POWER), W88.
- new net: IND1. (P), MOT15. (PWR), W116.
- new net: MOT10. (PWR), MOT12. (PWR), W112.
- new net: MOT12. (PWR), MOT13. (PWR), W113.
- new net: MOT10. (PWR), MOT14. (PWR), W111.
- new net: ETH1. (POWER), VRM2. (5V/2A), W84.
- new net: A3. (Power), ETH1. (POWER), W89.
- new net: MOT1. (PWR), MOT2. (PWR), W105.
- new net: MOT2. (PWR), MOT3. (PWR), W106.
- new net: MOT3. (PWR), MOT4. (PWR), W107.
- new net: A3. (Power), IMU1. (RIO_PWM2), W47.
- no-connect marks 46 -> 47
