File: robots/2024/system-drawing/kicad-schematic/2024-SystemDiagram.kicad_sch (KiCad schematic)
At the start: 180 parts

Commit message: Updated system drawing
Signed-off-by: Scott Berman <sgberman1@gmail.com>
Parts:
- added W118: BB_CAN_PWR, symbol SystemDiagram:WireTag
- W24: MFG (none) -> Automaton Direct
- renumbered A1 to NX1, A2 to NX2, A3 to NX3
Connections:
- net at POE1. (RJ45S): now also RDO1. (POWER); no longer VRM1. (5V/2A)
- net at RDO1. (POWER): now also ETH1. (POWER); no longer VRM1. (5V/2A)
- net at ETH1. (POWER): now also NX1. (Power), W87.; no longer RDO1. (POWER)
- new net: VRM1. (5V/2A), W118., WG1. (4)
- new net: POE1. (RJ45S), VRM1. (5V/2A)
- new net: RDO1. (POWER), VRM1. (5V/2A)
- new net: CAN1. (USB), W67., WG1. (4)
- new net: MOT7. (PWR), MOT8. (PWR), W108.
- new net: MOT8. (PWR), MOT9. (PWR), W109.
- new net: MOT11. (PWR), MOT13. (PWR), W114.
- new net: MOT11. (PWR), MOT15. (PWR), W115.
- new net: MOT14. (PWR), MOT9. (PWR), W110.
- new net: ETH1. (POWER), NX2. (Power), W88.
- new net: IND1. (P), MOT15. (PWR), W116.
- new net: MOT10. (PWR), MOT12. (PWR), W112.
- new net: MOT12. (PWR), MOT13. (PWR), W113.
- new net: MOT10. (PWR), MOT14. (PWR), W111.
- new net: ETH1. (POWER), VRM2. (5V/2A), W84.
- new net: ETH1. (POWER), NX3. (Power), W89.
- new net: MOT1. (PWR), MOT2. (PWR), W105.
- new net: MOT2. (PWR), MOT3. (PWR), W106.
- new net: MOT3. (PWR), MOT4. (PWR), W107.
- new net: IMU1. (RIO_PWM2), NX3. (Power), W47.
- no-connect marks 47 -> 69
Changed lines of the file:
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@@
   (junction (at 171.45 462.28) (diameter 0) (color 0 0 0 0)
   )
+  (junction (at 224.79 345.44) (diameter 0) (color 0 0 0 0)
+  )
   (junction (at 586.74 144.78) (diameter 0) (color 0 0 0 0)
   )
@@
   )
   (no_connect (at 224.79 452.12))
+  (no_connect (at 220.98 269.24))
   (no_connect (at 220.98 219.71))
   (no_connect (at 87.63 274.32))
@@
   (no_connect (at 224.79 434.34))
   (no_connect (at 605.79 129.54))
+  (no_connect (at 179.07 252.73))
+  (no_connect (at 179.07 257.81))
   (no_connect (at 220.98 227.33))
   (no_connect (at 87.63 266.7))
   (no_connect (at 605.79 142.24))
+  (no_connect (at 220.98 280.67))
   (no_connect (at 220.98 222.25))
   (no_connect (at 220.98 229.87))
+  (no_connect (at 208.28 353.06))
+  (no_connect (at 220.98 293.37))
+  (no_connect (at 179.07 269.24))
+  (no_connect (at 179.07 264.16))
   (no_connect (at 224.79 426.72))
   (no_connect (at 87.63 264.16))
@@
   (no_connect (at 224.79 401.32))
   (no_connect (at 191.77 401.32))
+  (no_connect (at 179.07 261.62))
   (no_connect (at 220.98 205.74))
   (no_connect (at 87.63 259.08))
   (no_connect (at 220.98 217.17))
+  (no_connect (at 220.98 288.29))
+  (no_connect (at 220.98 283.21))
+  (no_connect (at 208.28 363.22))
   (no_connect (at 220.98 208.28))
   (no_connect (at 224.79 436.88))
@@
   (no_connect (at 224.79 429.26))
   (no_connect (at 220.98 264.16))
+  (no_connect (at 179.07 228.6))
   (no_connect (at 191.77 434.34))
   (no_connect (at 224.79 398.78))
   (no_connect (at 191.77 472.44))
   (no_connect (at 191.77 436.88))
+  (no_connect (at 220.98 271.78))
+  (no_connect (at 208.28 360.68))
   (no_connect (at 224.79 469.9))
   (no_connect (at 224.79 328.93))
+  (no_connect (at 179.07 266.7))
+  (no_connect (at 220.98 298.45))
   (no_connect (at 224.79 457.2))
   (no_connect (at 220.98 200.66))
   (no_connect (at 220.98 495.3))
   (no_connect (at 220.98 261.62))
+  (no_connect (at 179.07 231.14))
   (no_connect (at 220.98 254))
+  (no_connect (at 220.98 295.91))
+  (no_connect (at 208.28 355.6))
+  (no_connect (at 220.98 285.75))
   (no_connect (at 87.63 279.4))
   (no_connect (at 224.79 472.44))
+  (no_connect (at 220.98 290.83))
   (no_connect (at 224.79 391.16))
   (no_connect (at 87.63 281.94))
@@
     (stroke (width 0.508) (type default) (color 255 0 0 1))
   )
-  (wire (pts (xy 208.28 345.44) (xy 256.54 345.44))
+  (wire (pts (xy 208.28 345.44) (xy 224.79 345.44))
     (stroke (width 0.254) (type default) (color 255 0 0 1))
   )
@@
     (stroke (width 0.508) (type default) (color 255 0 0 1))
   )
+  (wire (pts (xy 224.79 345.44) (xy 256.54 345.44))
+    (stroke (width 0.254) (type default) (color 255 0 0 1))
+  )
   (wire (pts (xy 237.49 232.41) (xy 220.98 232.41))
     (stroke (width 0.254) (type default) (color 194 0 194 1))
@@
   (symbol (lib_id "SystemDiagram:Orin_NX") (at 208.28 412.75 0) (unit 1)
     (in_bom yes) (on_board yes) (dnp no)
-    (property "Reference" "A2" (at 208.28 408.94 0)
+    (property "Reference" "NX2" (at 208.28 408.94 0)
       (effects (font (size 1.27 1.27)))
     )
@@
       (project "2024-SystemDiagram"
         (path "/12a52703-e3f4-4774-b510-3055ab1abf35"
-          (reference "A2") (unit 1)
+          (reference "NX2") (unit 1)
         )
       )
@@
       (effects (font (size 1.27 1.27)) hide)
     )
-    (property "Datasheet" "" (at 586.74 340.36 0)
+    (property "Datasheet" "Components/AutomationDirect-m8sensorcbl.pdf" (at 586.74 340.36 0)
       (effects (font (size 1.27 1.27)) hide)
     )
@@
     )
   )
+  (symbol (lib_id "SystemDiagram:WireTag") (at 224.79 345.44 0) (unit 1)
+    (in_bom yes) (on_board yes) (dnp no)
+    (property "Reference" "W118" (at 234.95 344.17 0)
+      (effects (font (size 1.27 1.27)))
+    )
+    (property "Value" "BB_CAN_PWR" (at 224.79 342.9 0)
+      (effects (font (size 1.27 1.27)))
+    )
+    (property "Footprint" "" (at 224.79 345.44 0)
+      (effects (font (size 1.27 1.27)) hide)
+    )
+    (property "Datasheet" "" (at 224.79 345.44 0)
+      (effects (font (size 1.27 1.27)) hide)
+    )
+    (pin "")
+    (instances
+      (project "2024-SystemDiagram"
+        (path "/12a52703-e3f4-4774-b510-3055ab1abf35"
+          (reference "W118") (unit 1)
+        )
+      )
+    )
+  )
   (symbol (lib_id "SystemDiagram:WireTag") (at 157.48 107.95 90) (unit 1)
     (in_bom yes) (on_board yes) (dnp no)
@@
       (effects (font (size 1.27 1.27)) hide)
     )
-    (property "Datasheet" "" (at 594.36 176.53 0)
+    (property "Datasheet" "Components/AutomationDirect-m8sensorcbl.pdf" (at 594.36 176.53 0)
       (effects (font (size 1.27 1.27)) hide)
     )
+    (property "MFG" "Automaton Direct" (at 593.09 179.07 0)
+      (effects (font (size 1.27 1.27)))
+    )
+    (property "MFG P/N" "" (at 593.09 181.61 0)
+      (effects (font (size 1.27 1.27)))
+    )
     (pin "")
     (instances
@@
       (effects (font (size 1.27 1.27)) hide)
     )
-    (property "Datasheet" "https://cdn.automationdirect.com/static/specs/peminirectqm.pdf" (at 622.3 444.5 0)
+    (property "Datasheet" "Components/AutomationDirect-BeamBreak.pdf" (at 622.3 444.5 0)
       (effects (font (size 1.27 1.27)) hide)
     )
@@
   (symbol (lib_id "SystemDiagram:Orin_NX") (at 208.28 448.31 0) (unit 1)
     (in_bom yes) (on_board yes) (dnp no)
-    (property "Reference" "A3" (at 208.28 444.5 0)
+    (property "Reference" "NX3" (at 208.28 444.5 0)
       (effects (font (size 1.27 1.27)))
     )
@@
       (project "2024-SystemDiagram"
         (path "/12a52703-e3f4-4774-b510-3055ab1abf35"
-          (reference "A3") (unit 1)
+          (reference "NX3") (unit 1)
         )
       )
@@
   (symbol (lib_id "SystemDiagram:Orin_NX") (at 208.28 377.19 0) (unit 1)
     (in_bom yes) (on_board yes) (dnp no)
-    (property "Reference" "A1" (at 208.28 373.38 0)
+    (property "Reference" "NX1" (at 208.28 373.38 0)
       (effects (font (size 1.27 1.27)))
     )
@@
       (project "2024-SystemDiagram"
         (path "/12a52703-e3f4-4774-b510-3055ab1abf35"
-          (reference "A1") (unit 1)
+          (reference "NX1") (unit 1)
         )
       )
@@
       (effects (font (size 1.27 1.27)) hide)
     )
-    (property "Datasheet" "" (at 590.55 440.69 0)
+    (property "Datasheet" "Components/AutomationDirect-m8sensorcbl.pdf" (at 590.55 440.69 0)
       (effects (font (size 1.27 1.27)) hide)
     )
@@
       (effects (font (size 1.27 1.27)) hide)
     )
-    (property "Datasheet" "https://cdn.automationdirect.com/static/specs/peminirectqm.pdf" (at 623.57 344.17 0)
+    (property "Datasheet" "Components/AutomationDirect-BeamBreak.pdf" (at 623.57 344.17 0)
       (effects (font (size 1.27 1.27)) hide)
     )
@@
       (effects (font (size 1.27 1.27)) hide)
     )
-    (property "Datasheet" "https://cdn.automationdirect.com/static/specs/peminirectqm.pdf" (at 621.03 180.34 0)
+    (property "Datasheet" "Components/AutomationDirect-BeamBreak.pdf" (at 621.03 180.34 0)
       (effects (font (size 1.27 1.27)) hide)
     )

Commit message: Updated the motor can bus assignments
Signed-off-by: Scott Berman <sgberman1@gmail.com>
Parts:
- removed CAN5: CAN_Terminator, symbol SystemDiagram:CAN_Terminator
- removed W116: CAN, symbol SystemDiagram:WireTag
- added CAN101: CAN_Terminator, symbol SystemDiagram:CAN_Terminator
- added W119: CAN, symbol SystemDiagram:WireTag
Connections:
- net CAN_PD: now also MOT9. (PWR); no longer MOT7. (PWR)
- net at POE1. (RJ45S): now also RDO1. (POWER); no longer VRM1. (5V/2A)
- net at RDO1. (POWER): now also ETH1. (POWER); no longer VRM1. (5V/2A)
- net at ETH1. (POWER): now also NX1. (Power), W87.; no longer RDO1. (POWER)
- net at W117.: now also MOT7. (PWR), CAN101.; no longer IND1. (P)
- new net: VRM1. (5V/2A), W118., WG1. (4)
- new net: POE1. (RJ45S), VRM1. (5V/2A)
- new net: RDO1. (POWER), VRM1. (5V/2A)
- new net: CAN1. (USB), W67., WG1. (4)
- new net: IND1. (P), MOT11. (PWR), W114.
- new net: MOT11. (PWR), MOT13. (PWR), W113.
- new net: ETH1. (POWER), NX2. (Power), W88.
- new net: MOT10. (PWR), MOT12. (PWR), W111.
- new net: MOT12. (PWR), MOT13. (PWR), W112.
- new net: IND1. (P), MOT15. (PWR), W115.
- new net: ETH1. (POWER), VRM2. (5V/2A), W84.
- new net: ETH1. (POWER), NX3. (Power), W89.
- new net: MOT1. (PWR), MOT2. (PWR), W105.
- new net: MOT2. (PWR), MOT3. (PWR), W106.
- new net: CAN4., MOT14. (PWR), W110.
- new net: MOT3. (PWR), MOT4. (PWR), W107.
- new net: IMU1. (RIO_PWM2), NX3. (Power), W47.
- new net CAN_ALT_TO_NOTE_RET: MOT15. (PWR), MOT7. (PWR), W108.
- new net CAN_FD_DRV_TURRET: MOT4. (PWR), MOT8. (PWR), W104.
- new net CAN_FD_TURRET_INTAKE_PIVOT: MOT14. (PWR), MOT8. (PWR), W119.
- new net CAN_INTAKE_TO_XFR_ROLLER: MOT10. (PWR), MOT9. (PWR), W109.
Other:
- moved on the sheet: CAN4, W108, W27, W28
