File: tools/CNC-router/RouterEstop/RouterEstop.kicad_sch (KiCad schematic)
At the start: 36 parts, among them J1 OUT4, J2 OUT7, J3 IN13, K2 K2, K3 K_{m}, K4 BRAKE, K5 DRIVE_INHIBIT, SW1 ON, SW2 OFF, SW3 ESTOP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

Commit message: Update CNC router to as-built
Signed-off-by: Scott <sgberman1@gmail.com>
Parts:
- removed unit 2 of K2
- added D4: RED, symbol Device:LED
- added D5: GREEN, symbol Device:LED
- added J4: OUT3, symbol Connector:Screw_Terminal_01x02
- added J5: OUT5, symbol Connector:Screw_Terminal_01x02
- K1: value ~ -> K1
Connections:
- net 24V: now also D4.2 (A), D5.2 (A)
- net RTN: now also J4.- (Pin_2), J5.- (Pin_2)
- net at J2.+ (Pin_1), SW5.2 (B), TP7.1: now also J3.+ (Pin_1)
- new net: D5.1 (K), J5.+ (Pin_1)
- new net: D4.1 (K), J4.+ (Pin_1)
Other:
- note added: "STACK LIGHT"
