File: circuit-boards/Orin-NX-PCBs/NX-IndicatorBoard/LEDs.kicad_sch (KiCad schematic)
At the start: 55 parts, among them Q1 BSS138W, Q10 BSS138W, Q11 BSS138W, Q12 BSS138W, Q13 BSS138W, Q14 BSS138W, Q2 BSS138W, Q3 BSS138W, Q4 BSS138W, Q5 BSS138W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

Commit message: Intermediate checkin of NX-Indicator-board
Signed-off-by: Scott Berman <scott.berman@bluerivertech.com>
Parts:
- R21: now not fitted
Other:
- note added: "NOTE: PULL DOWN RESITORS MUST BE GREATER THAN 50k TO COMPLY WITH LEVEL TRANSLATOR"
