File: circuit-boards/Orin-NX-PCBs/NX-IndicatorBoard-V2/LEDs.kicad_sch (KiCad schematic)
At the start: 22 parts, among them U1 74LVC245ABQ

Commit message: Check in of NX Adapter and Indicator boards.  Complete pending review
Signed-off-by: Scott <sgberman1@gmail.com>
Parts:
- C5: value 0.1uF-10%-50V-0603 -> 0.1uF-10%-50V-0805; footprint Capacitor_SMD:C_0603_1608Metric -> Capacitor_SMD:C_0805_2012Metric; DIST P/N 1276-1000-1-ND -> 311-1140-1-ND; MFG Samsung Electro-Mechanics -> YAGEO; MFG P/N CL10B104KB8NNNC -> CC0805KRX7R9BB104
- R1, R2, R3, R4, R5, R6, R7, R8: value 499R-1%-0603 -> 499R-1%-0805; footprint Resistor_SMD:R_0603_1608Metric -> Resistor_SMD:R_0805_2012Metric; DIST P/N 311-499HRCT-ND -> 311-499CRCT-ND; MFG P/N RC0603FR-07499RL -> RC0805FR-07499RL
- renumbered D3 to D1, D4 to D2, D5 to D3, D6 to D4, D7 to D5, D8 to D6, D9 to D7, D10 to D8, D11 to D9

Commit message: Intermediate checkin of NX-Indicator-board
Signed-off-by: Scott Berman <scott.berman@bluerivertech.com>
Parts:
- removed D2: ETH, LED_SMD:LED_1206_3216Metric, symbol Device:LED
- removed D4: USR1, LED_SMD:LED_1206_3216Metric, symbol Device:LED
- removed D7: USR2, LED_SMD:LED_1206_3216Metric, symbol Device:LED
- removed LP1, LP2, LP3: Lumex-3x-Light-Pipe, NX-IndicatorBoard:LUMEX-LPF-C013301S, symbol NX-IndicatorBoard:Lumex-3x-Light-Pipe
- removed R1, R2, R5: 499R-1%-0805, Resistor_SMD:R_0805_2012Metric, symbol Device:R_US
- added LP1, LP2, LP3: Lumex-2x-Light-Pipe, NX-IndicatorBoard:Lumex-LPF-C012303S, symbol NX-IndicatorBoard:Lumex-2x-Light-Pipe
Connections:
- no-connect marks 0 -> 3
Other:
- note added: "CPU CAN2"
- note added: "HD CAN1"
- note added: "PC CAN0"
- note removed: "CAN0 CAN1 CAN2"
- note removed: "ETH HD CPU"
- note removed: "PC USR1 USR2"

Commit message: Checkin of NX Indicator board 2x CAN FD + 6 LEDs
Signed-off-by: Scott <sgberman1@gmail.com>
Parts:
- renumbered D8 to D3, D5 to D4, D1 to D5, D9 to D6, D6 to D7, D3 to D8, LP3 to LP1, LP1 to LP3, R4 to R1, R8 to R2, R7 to R3, R6 to R4, R3 to R5
Connections:
- net ETH is gone; now on net GND: U1.5 (A3)
- net USR1 is gone; now on net GND: U1.8 (A6)
- net USR2 is gone; now on net GND: U1.9 (A7)

Commit message: Fix bom. Made LVC245 an SO-20 part
Signed-off-by: Scott Berman <scott.berman@bluerivertech.com>
Parts:
- U1: value 74LVC245ABQ -> 74LVC245AD; DIST P/N 1727-3495-1-ND -> 1727-3104-1-ND; MFG P/N 74LVC245ABQ,115 -> 74LVC245AD,118
Changed lines of the file:
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@@
 	(title_block
 		(title "NX Indicator Board V2")
-		(date "2024-07-28")
+		(date "2024-08-05")
 		(rev "2")
 		(company "971 Spartan Robotics")
@@
 			)
 		)
-		(property "Value" "74LVC245ABQ"
+		(property "Value" "74LVC245AD"
 			(at 186.3441 115.57 0)
 			(effects
@@
 			)
 		)
-		(property "MFG P/N" "74LVC245ABQ,115"
+		(property "MFG P/N" "74LVC245AD,118"
 			(at 184.15 133.35 0)
 			(effects
@@
 			)
 		)
-		(property "DIST P/N" "1727-3495-1-ND"
+		(property "DIST P/N" "1727-3104-1-ND"
 			(at 184.15 133.35 0)
 			(effects
