File: circuit-boards/Orin-NX-PCBs/NX-J401-Adapter-v3/nx-can.kicad_sch (KiCad schematic)
At the start: 9 parts, among them U2 MCP2542FDT-E/SN, U3 TPS613222ADBVR

Commit message: NX Adapter interim checking
Signed-off-by: Scott <sgberman1@gmail.com>
Parts:
- removed C24 (x2): 0.1uF-10%-50V-0603, Capacitor_SMD:C_0603_1608Metric, symbol Device:C
- removed C? (x2): 22uF-20%-0603, Capacitor_SMD:C_0603_1608Metric, symbol Device:C
- added C10, C14: 0.22uF-10%-50V-0805, Capacitor_SMD:C_0805_2012Metric, symbol Device:C
- added C11, C13: 22uF-20%-25V-0805, Capacitor_SMD:C_0805_2012Metric, symbol Device:C
Connections:
- net +5V: now also C10.1, C11.1, C13.1
- net 3V3: now also C14.1
- net GNDD: now also C10.2, C11.2, C13.2, C14.2

Commit message: Check in of NX Adapter and Indicator boards.  Complete pending review
Signed-off-by: Scott <sgberman1@gmail.com>
Parts:
- D7: DIST (none) -> Digkey; DIST P/N (none) -> 1727-3817-1-ND
- U1: renamed from U2; value MCP2542FDT-E/SN -> MCP2558FD-H/SN; DIST P/N MCP2542FDT-E/SNCT-ND -> MCP2558FD-H/SN-ND; MFG P/N MCP2542FDT-E/SN -> MCP2558FD-H/SN
- renumbered C13 to C10, C10 to C3, C14 to C4, C11 to C9
Changed lines of the file:
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@@
 			(project "IMU-2X"
 				(path "/cc31ce4b-09ab-4aea-a1d3-ed84696ba658/b82ca404-386f-4bdf-8b2c-60800790d9b9"
-					(reference "L2")
+					(reference "L1")
 					(unit 1)
 				)
@@
 			)
 		)
+		(property "DIST" "Digkey"
+			(at 245.11 104.14 0)
+			(effects
+				(font
+					(size 1.27 1.27)
+				)
+				(hide yes)
+			)
+		)
+		(property "DIST P/N" "1727-3817-1-ND"
+			(at 245.11 104.14 0)
+			(effects
+				(font
+					(size 1.27 1.27)
+				)
+				(hide yes)
+			)
+		)
 		(pin "1"
 		)
@@
 			(project "PI-Power-Board"
 				(path "/cc31ce4b-09ab-4aea-a1d3-ed84696ba658/b82ca404-386f-4bdf-8b2c-60800790d9b9"
-					(reference "D5")
+					(reference "D2")
 					(unit 1)
 				)
@@
 		(on_board yes)
 		(dnp no)
-		(property "Reference" "C13"
+		(property "Reference" "C10"
 			(at 232.41 175.26 0)
 			(effects
@@
 			(project "NX-J401-Adapter"
 				(path "/cc31ce4b-09ab-4aea-a1d3-ed84696ba658/b82ca404-386f-4bdf-8b2c-60800790d9b9"
-					(reference "C13")
+					(reference "C10")
 					(unit 1)
 				)
@@
 		(on_board yes)
 		(dnp no)
-		(property "Reference" "C14"
+		(property "Reference" "C4"
 			(at 194.31 70.866 0)
 			(effects
@@
 			)
 		)
-		(property "Datasheet" "~"
+		(property "Datasheet" "Components/KEMET_C1002_X7R_SMD.pdf"
 			(at 195.58 73.66 0)
 			(effects
@@
 			(project "NX-J401-Adapter"
 				(path "/cc31ce4b-09ab-4aea-a1d3-ed84696ba658/b82ca404-386f-4bdf-8b2c-60800790d9b9"
-					(reference "C14")
+					(reference "C4")
 					(unit 1)
 				)
@@
 		(on_board yes)
 		(dnp no)
-		(property "Reference" "C11"
+		(property "Reference" "C9"
 			(at 245.11 175.26 0)
 			(effects
@@
 			(project "NX-J401-Adapter"
 				(path "/cc31ce4b-09ab-4aea-a1d3-ed84696ba658/b82ca404-386f-4bdf-8b2c-60800790d9b9"
-					(reference "C11")
+					(reference "C9")
 					(unit 1)
 				)
@@
 		(on_board yes)
 		(dnp no)
-		(property "Reference" "C10"
+		(property "Reference" "C3"
 			(at 209.55 70.866 0)
 			(effects
@@
 			)
 		)
-		(property "Datasheet" "~"
+		(property "Datasheet" "Components/KEMET_C1002_X7R_SMD.pdf"
 			(at 208.28 73.66 0)
 			(effects
@@
 			(project "NX-J401-Adapter"
 				(path "/cc31ce4b-09ab-4aea-a1d3-ed84696ba658/b82ca404-386f-4bdf-8b2c-60800790d9b9"
-					(reference "C10")
+					(reference "C3")
 					(unit 1)
 				)
@@
 			(project "IMU-2X"
 				(path "/cc31ce4b-09ab-4aea-a1d3-ed84696ba658/b82ca404-386f-4bdf-8b2c-60800790d9b9"
-					(reference "C9")
+					(reference "C8")
 					(unit 1)
 				)
@@
 		(on_board yes)
 		(dnp no)
-		(property "Reference" "U2"
+		(property "Reference" "U1"
 			(at 209.55 83.82 0)
 			(effects
@@
 			)
 		)
-		(property "Value" "MCP2542FDT-E/SN"
+		(property "Value" "MCP2558FD-H/SN"
 			(at 207.01 101.6 0)
 			(effects
@@
 			)
 		)
-		(property "Datasheet" "Components/Microchip-MCP2542WFD.pdf"
+		(property "Datasheet" "Components/Microchip-MCP2558.pdf"
 			(at 203.2 92.71 0)
 			(effects
@@
 			)
 		)
-		(property "MFG P/N" "MCP2542FDT-E/SN"
+		(property "MFG P/N" "MCP2558FD-H/SN"
 			(at 203.2 92.71 0)
 			(effects
@@
 			)
 		)
-		(property "DIST P/N" "MCP2542FDT-E/SNCT-ND"
+		(property "DIST P/N" "MCP2558FD-H/SN-ND"
 			(at 203.2 92.71 0)
 			(effects
@@
 			(project "NX-J401-Adapter"
 				(path "/cc31ce4b-09ab-4aea-a1d3-ed84696ba658/b82ca404-386f-4bdf-8b2c-60800790d9b9"
-					(reference "U2")
-					(unit 1)
-				)
+					(reference "U1")
+					(unit 1)
+				)

Commit message: Minor update to NX-J401-Adapter-v3
Signed-off-by: Scott Berman <scott.berman@bluerivertech.com>
Changed lines of the file:
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@@
 	(title_block
 		(title "NX J401 Adapter")
-		(rev "1")
+		(date "2024-08-05")
+		(rev "3")
 		(company "971 Spartan Robotics")
 	)
@@
 	(symbol
 		(lib_id "Graphic:SYM_Arrow_Normal")
-		(at 182.88 147.32 0)
+		(at 173.99 204.47 0)
 		(unit 1)
 		(exclude_from_sim yes)
@@
 		(dnp no)
 		(property "Reference" "#SYM5"
-			(at 182.88 145.796 0)
+			(at 173.99 202.946 0)
 			(effects
 				(font
@@
 		)
 		(property "Value" "Boost Regulator Design Notes"
-			(at 186.69 147.32 0)
+			(at 177.8 204.47 0)
 			(effects
 				(font
@@
 				)
 				(justify left)
+				(hide yes)
 			)
 		)
 		(property "Footprint" ""
-			(at 182.88 147.32 0)
-			(effects
-				(font
-					(size 1.27 1.27)
-				)
-				(hide yes)
-			)
-		)
-		(property "Datasheet" "Components/WBDesign78-TPS613222-3Vin-5Vout-0.25A.pdf"
-			(at 182.88 147.32 0)
-			(effects
-				(font
-					(size 1.27 1.27)
-				)
-				(hide yes)
+			(at 173.99 204.47 0)
+			(effects
+				(font
+					(size 1.27 1.27)
+				)
+				(hide yes)
+			)
+		)
+		(property "Datasheet" "Analysis/WBDesign78-TPS613222-3Vin-5Vout-0.25A.pdf"
+			(at 177.165 204.47 0)
+			(effects
+				(font
+					(size 1.27 1.27)
+				)
+				(justify left)
 			)
 		)
 		(property "Description" ""
-			(at 182.88 147.32 0)
-			(effects
-				(font
+			(at 173.99 204.47 0)
+			(effects
+				(font

Commit message: Updated diff pairs and power supply layout
Signed-off-by: Scott <sgberman1@gmail.com>
Parts:
- renumbered C3 to C10, C10 to C11, C9 to C12, C4 to C13, U1 to U3
Changed lines of the file:
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@@
 	(title_block
 		(title "NX J401 Adapter")
-		(date "2024-08-05")
+		(date "2024-08-10")
 		(rev "3")
 		(company "971 Spartan Robotics")
@@
 			(project "IMU-2X"
 				(path "/cc31ce4b-09ab-4aea-a1d3-ed84696ba658/b82ca404-386f-4bdf-8b2c-60800790d9b9"
-					(reference "L1")
+					(reference "L2")
 					(unit 1)
 				)
@@
 			(project "PI-Power-Board"
 				(path "/cc31ce4b-09ab-4aea-a1d3-ed84696ba658/b82ca404-386f-4bdf-8b2c-60800790d9b9"
-					(reference "D2")
+					(reference "D4")
 					(unit 1)
 				)
@@
 		(on_board yes)
 		(dnp no)
-		(property "Reference" "C10"
+		(property "Reference" "C11"
 			(at 232.41 175.26 0)
 			(effects
@@
 			(project "NX-J401-Adapter"
 				(path "/cc31ce4b-09ab-4aea-a1d3-ed84696ba658/b82ca404-386f-4bdf-8b2c-60800790d9b9"
-					(reference "C10")
+					(reference "C11")
 					(unit 1)
 				)
@@
 			(project "IMU-2X"
 				(path "/cc31ce4b-09ab-4aea-a1d3-ed84696ba658/b82ca404-386f-4bdf-8b2c-60800790d9b9"
-					(reference "U3")
+					(reference "U2")
 					(unit 1)
 				)
@@
 		(on_board yes)
 		(dnp no)
-		(property "Reference" "C4"
+		(property "Reference" "C13"
 			(at 194.31 70.866 0)
 			(effects
@@
 			(project "NX-J401-Adapter"
 				(path "/cc31ce4b-09ab-4aea-a1d3-ed84696ba658/b82ca404-386f-4bdf-8b2c-60800790d9b9"
-					(reference "C4")
+					(reference "C13")
 					(unit 1)
 				)
@@
 		(on_board yes)
 		(dnp no)
-		(property "Reference" "C9"
+		(property "Reference" "C12"
 			(at 245.11 175.26 0)
 			(effects
@@
 			(project "NX-J401-Adapter"
 				(path "/cc31ce4b-09ab-4aea-a1d3-ed84696ba658/b82ca404-386f-4bdf-8b2c-60800790d9b9"
-					(reference "C9")
+					(reference "C12")
 					(unit 1)
 				)
@@
 		(on_board yes)
 		(dnp no)
-		(property "Reference" "C3"
+		(property "Reference" "C10"
 			(at 209.55 70.866 0)
 			(effects
@@
 			(project "NX-J401-Adapter"
 				(path "/cc31ce4b-09ab-4aea-a1d3-ed84696ba658/b82ca404-386f-4bdf-8b2c-60800790d9b9"
-					(reference "C3")
+					(reference "C10")
 					(unit 1)
 				)
@@
 			(project "IMU-2X"
 				(path "/cc31ce4b-09ab-4aea-a1d3-ed84696ba658/b82ca404-386f-4bdf-8b2c-60800790d9b9"
-					(reference "C8")
+					(reference "C9")
 					(unit 1)
 				)
@@
 		(on_board yes)
 		(dnp no)
-		(property "Reference" "U1"
+		(property "Reference" "U3"
 			(at 209.55 83.82 0)
 			(effects
@@
 			(project "NX-J401-Adapter"
 				(path "/cc31ce4b-09ab-4aea-a1d3-ed84696ba658/b82ca404-386f-4bdf-8b2c-60800790d9b9"
-					(reference "U1")
-					(unit 1)
-				)
+					(reference "U3")
+					(unit 1)
+				)
