File: circuit-boards/Orin-NX-PCBs/NX-ButtonInterface-v2/NX-ButtonInterface.kicad_pcb (KiCad board)
At the start: 2 copper layers, 48.3 x 21.2 mm, 3 parts, among them J1 NX CONTROL & UART, J2 NX-BUTTON, J4 POWER LED

Commit message: Add NX Button Interface V2
Signed-off-by: Scott <sgberman1@gmail.com>
Parts:
- moved J2 34.3 mm to (125.5, 109.6)
- moved J4 34.3 mm to (91.2, 104.9)
Connections:
- J2 pad 1: /CAN_TX -> /~{REC}
- J2 pad 2: /CAN_RX -> /SYS_RST_RCV_RTN
- J2 pad 3: /GND -> /~{SYS_RESET}
- J2 pad 4: /3V3 -> /UART2_TXD
- J2 pad 6: /UART2_TXD -> /3V3
- J2 pad 7: /~{SYS_RESET} -> /GND
- J2 pad 8: /SYS_RST_RCV_RTN -> /CAN_RX
- J2 pad 9: /~{REC} -> /CAN_TX
- J4 pad 1: /NX_PC_LED- -> /NX_PC_LED+
- J4 pad 2: /NX_PC_LED+ -> /NX_PC_LED-
Routing:
- net /~{REC}: track 4.16 -> 40.5 mm, vias 0 -> 1
- net /CAN_RX: track 42.9 -> 7.38 mm, vias 2 -> 0
- net /CAN_TX: track 45.8 -> 11.4 mm, vias 1 -> 0
- net /SYS_RST_RCV_RTN: track 20.5 -> 43.9 mm
- net /~{SYS_RESET}: track 15.3 -> 34.1 mm, vias 0 -> 1
- net /NX_PC_LED+: track 50.1 -> 32.2 mm, vias 1 -> 0
- net /3V3: track 36.1 -> 21.3 mm, vias 2 -> 0
- net /NX_PC_LED-: track 50.9 -> 37.7 mm, vias 1 -> 0
- net /GND: track 11.6 -> 19.8 mm
- net /UART2_TXD: track 19.4 -> 25.2 mm
- net /UART2_RXD: track 22.6 -> 21.7 mm, vias 0 -> 1
- removed copper zone on B.Cu, net /GND
Other:
- board text added: "1 ~{REC}"
- board text added: "3 ~{RESET}"
- board text added: "3V3 6"
- board text added: "5 RXD"
- board text added: "7 GND"
- board text added: "9 CAN TX"
- board text added: "CAN RX 8"
- board text added: "LED+ 1"
- board text added: "LED- 2"
- board text added: "RTN 2"
- board text added: "SPARTAN ROBOTICS 2024 NX BUTTON INTERFACE V2"
- board text added: "TXD 4"
- board text removed: "1 LED-"
- board text removed: "2 CAN RX"
- board text removed: "2 LED+"
- board text removed: "4 3V3"
- board text removed: "6 TXD"
- board text removed: "8 RTN"
- board text removed: "CAN TX 1"
- board text removed: "GND 3"
- board text removed: "NX BUTTON INTERFACE V2 SPARTAN ROBOTICS 2024"
- board text removed: "RXD 5"
- board text removed: "~{REC} 9"
- board text removed: "~{RESET} 7"
