File: circuit-boards/Orin-NX-PCBs/NX-ButtonInterface-v2/NX-ButtonInterface.kicad_sch (KiCad schematic)
At the start: 3 parts, among them J1 NX CONTROL & UART, J2 NX-BUTTON, J4 POWER LED

Commit message: Add NX Button Interface V2
Signed-off-by: Scott <sgberman1@gmail.com>
Connections:
- net 3V3: now also J2.6 (Pin_6); no longer J2.4 (Pin_4)
- net CAN_RX: now also J2.8 (Pin_8); no longer J2.2 (Pin_2)
- net CAN_TX: now also J2.9 (Pin_9); no longer J2.1 (Pin_1)
- net GND: now also J2.7 (Pin_7); no longer J2.3 (Pin_3)
- net NX_PC_LED+: now also J4.1 (Pin_1); no longer J4.2 (Pin_2)
- net NX_PC_LED-: now also J4.2 (Pin_2); no longer J4.1 (Pin_1)
- net SYS_RST_RCV_RTN: now also J2.2 (Pin_2); no longer J2.8 (Pin_8)
- net UART2_TXD: now also J2.4 (Pin_4); no longer J2.6 (Pin_6)
- net ~{REC}: now also J2.1 (Pin_1); no longer J2.9 (Pin_9)
- net ~{SYS_RESET}: now also J2.3 (Pin_3); no longer J2.7 (Pin_7)
Other:
- company: (none) -> 971 SPARTAN ROBOTICS
- title: Button Interface -> NX Button Interface V2
Changed lines of the file:
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@@
 	(paper "A")
 	(title_block
-		(title "Button Interface")
-		(date "2024-01-05")
+		(title "NX Button Interface V2")
+		(date "2024-08-16")
 		(rev "1")
+		(company "971 SPARTAN ROBOTICS")
 	)
 	(no_connect
@@
 		)
 	)
-	(label "~{REC}"
-		(at 166.37 99.06 180)
-		(fields_autoplaced yes)
-		(effects
-			(font
-				(size 1.27 1.27)
-			)
-			(justify right bottom)
-		)
-	)
-	(label "CAN_TX"
-		(at 166.37 78.74 180)
+	(label "NX_PC_LED-"
+		(at 166.37 68.58 180)
+		(fields_autoplaced yes)
+		(effects
+			(font
+				(size 1.27 1.27)
+			)
+			(justify right bottom)
+		)
+	)
+	(label "UART2_TXD"
+		(at 166.37 86.36 180)
 		(fields_autoplaced yes)
 		(effects
@@
 		)
 	)
+	(label "GND"
+		(at 95.25 77.47 0)
+		(fields_autoplaced yes)
+		(effects
+			(font
+				(size 1.27 1.27)
+			)
+			(justify left bottom)
+		)
+	)
+	(label "3V3"
+		(at 166.37 91.44 180)
+		(fields_autoplaced yes)
+		(effects
+			(font
+				(size 1.27 1.27)
+			)
+			(justify right bottom)
+		)
+	)
+	(label "~{REC}"
+		(at 95.25 110.49 0)
+		(fields_autoplaced yes)
+		(effects
+			(font
+				(size 1.27 1.27)
+			)
+			(justify left bottom)
+		)
+	)
 	(label "UART2_RXD"
 		(at 166.37 88.9 180)
@@
 		)
 	)
-	(label "GND"
-		(at 95.25 77.47 0)
-		(fields_autoplaced yes)
-		(effects
-			(font
-				(size 1.27 1.27)
-			)
-			(justify left bottom)
-		)
-	)
-	(label "UART2_TXD"
-		(at 166.37 91.44 180)
-		(fields_autoplaced yes)
-		(effects
-			(font
-				(size 1.27 1.27)
-			)
-			(justify right bottom)
-		)
-	)
-	(label "~{REC}"
-		(at 95.25 110.49 0)
-		(fields_autoplaced yes)
-		(effects
-			(font
-				(size 1.27 1.27)
-			)
-			(justify left bottom)
-		)
-	)
-	(label "3V3"
-		(at 166.37 86.36 180)
-		(fields_autoplaced yes)
-		(effects
-			(font
-				(size 1.27 1.27)
-			)
-			(justify right bottom)
-		)
-	)
 	(label "NX_PC_LED+"
 		(at 95.25 90.17 0)
@@
 		)
 	)
-	(label "GND"
-		(at 166.37 83.82 180)
+	(label "SYS_RST_RCV_RTN"
+		(at 166.37 81.28 180)
+		(fields_autoplaced yes)
+		(effects
+			(font
+				(size 1.27 1.27)
+			)
+			(justify right bottom)
+		)
+	)
+	(label "CAN_TX"
+		(at 166.37 99.06 180)
 		(fields_autoplaced yes)
 		(effects
@@
 		)
 	)
-	(label "NX_PC_LED-"
-		(at 166.37 66.04 180)
+	(label "CAN_RX"
+		(at 166.37 96.52 180)
+		(fields_autoplaced yes)
+		(effects
+			(font
+				(size 1.27 1.27)
+			)
+			(justify right bottom)
+		)
+	)
+	(label "~{SYS_RESET}"
+		(at 166.37 83.82 180)
 		(fields_autoplaced yes)
 		(effects
@@
 		)
 	)
-	(label "SYS_RST_RCV_RTN"
-		(at 166.37 96.52 180)
-		(fields_autoplaced yes)
-		(effects
-			(font
-				(size 1.27 1.27)
-			)
-			(justify right bottom)
-		)
-	)
-	(label "CAN_RX"
-		(at 166.37 81.28 180)
+	(label "GND"
+		(at 166.37 93.98 180)
 		(fields_autoplaced yes)
 		(effects
@@
 	)
 	(label "NX_PC_LED+"
-		(at 166.37 68.58 180)
+		(at 166.37 66.04 180)
+		(fields_autoplaced yes)
+		(effects
+			(font
+				(size 1.27 1.27)
+			)
+			(justify right bottom)
+		)
+	)
+	(label "~{REC}"
+		(at 166.37 78.74 180)
 		(fields_autoplaced yes)
 		(effects
@@
 		)
 	)
-	(label "~{SYS_RESET}"
-		(at 166.37 93.98 180)
-		(fields_autoplaced yes)
-		(effects
-			(font
-				(size 1.27 1.27)
-			)
-			(justify right bottom)
-		)
-	)
