File: circuit-boards/shaft-encoders/mag-encoder2/mag-encoder.kicad_pcb (KiCad board)
At the start: 4 copper layers, 26.7 x 31.8 mm, 23 parts, among them J1 0015912055, J2 CONFIG, U1 AP2120N-3.3TRG1, U2 SN74LVC1G02DBVR, U3 MA732GQ

Commit message: Checking in 2 options of mag-encoder.  WIP
Signed-off-by: Scott <sgberman1@gmail.com>
Parts:
- D1: renamed from D5; value PWR -> ON
- D3: renamed from D2; value LOW -> LO
- D4: value HIGH -> HI
- moved D3 26.3 mm to (213.2, 119.5)
- moved D2 25.3 mm to (211.5, 119.5)
- moved D1 23.6 mm to (209.7, 119.5)
- moved D4 20.2 mm to (215.0, 119.5), turned to 90 degrees
- moved R6 16.9 mm to (217.6, 113.4), turned to -90 degrees
- moved R7 16.4 mm to (216.0, 113.4)
- moved R5 14.8 mm to (219.1, 113.4), turned to -90 degrees
- moved R4 12.5 mm to (220.6, 113.4)
- moved C1 3.14 mm to (226.9, 113.2), turned to -90 degrees
- moved U2 1.05 mm to (228.9, 109.6), turned to 90 degrees
- moved D5 0.67 mm to (228.9, 113.8), turned to -90 degrees
- moved C2 0.51 mm to (228.1, 106.0)
- moved H2 0.10 mm to (223.9, 117.5)
- renumbered C2 to C1, C1 to C2, D3 to D2, D1 to D5, H3 to H1, H4 to H2, H1 to H3, H2 to H4, R5 to R1, R6 to R2, R7 to R3, R2 to R4, R4 to R5, R1 to R6, R3 to R7, U2 to U1, U1 to U2
Routing:
- net Net-(U3-MGH): track 11.3 -> 23.0 mm
- net Net-(U3-MGL): track 7.45 -> 19.0 mm
- net Net-(R6-Pad1): track 8.02 -> 17.9 mm, vias 1 -> 2
- net Net-(D1-K): track 1.82 -> 11.4 mm
- net Net-(D2-A): track 2.99 -> 9.68 mm
- net Net-(D4-A): track 2.72 -> 9.09 mm
- net Net-(D3-A): track 3.91 -> 9.48 mm
- net +3.3V: track 8.90 -> 12.9 mm, vias 2 -> 3
- net GND: track 22.2 -> 24.0 mm, vias 7 -> 9
- net +5V_IN: track 12.6 -> 10.8 mm, vias 0 -> 2
- net /MOSI: track 23.0 -> 24.3 mm
- net /SCLK: track 16.9 -> 17.8 mm
- net Net-(U3-B): track 5.53 -> 6.11 mm
Other:
- board size 26.7 x 31.8 mm -> 24.1 x 31.8 mm
- board text added: "MAG ENCODER V1 971 SPARTAN ROBOTICS 2024"
- board text removed: "971 SPARTAN ROBOTICS 2024 MAG ENCODER V1"
