File: circuit-boards/shaft-encoders/mag-encoder3/mag-encoder.kicad_pcb (KiCad board)
At the start: 4 copper layers, 26.7 x 31.8 mm, 23 parts, among them J1 0015912055, J2 CONFIG, U1 AP2120N-3.3TRG1, U2 SN74LVC1G02DBVR, U3 MA732GQ

Commit message: Checking in 2 options of mag-encoder.  WIP
Signed-off-by: Scott <sgberman1@gmail.com>
Parts:
- removed H3: Pin, mag-encoder:pin-0.100
- removed H4: Slot, mag-encoder:slot-0.100x0.120
- added C1: 1uF-10%-25V-0603, Capacitor_SMD:C_0603_1608Metric, B.Cu at (237.3, 135.4)
- added C4: 1uF-10%-25V-0603, Capacitor_SMD:C_0603_1608Metric, B.Cu at (223.4, 111.5)
- C2: renamed from C1; moved to B.Cu
- C3: renamed from C2; moved to B.Cu
- D1: renamed from D5; value PWR -> ON
- D4: renamed from D2; value LOW -> LO
- D5: renamed from D4; value HIGH -> HI
- moved H2 41.7 mm to (230.6, 136.3), turned to 180 degrees
- moved J2 37.5 mm to (241.5, 123.6), turned to 90 degrees
- moved D4 34.8 mm to (224.5, 135.4)
- moved U2 34.1 mm to (237.3, 135.4), turned to 90 degrees
- moved D2 31.5 mm to (222.9, 135.4)
- moved R1 29.0 mm to (237.3, 133.9), turned to 180 degrees
- moved R5 28.6 mm to (226.1, 130.7), turned to 180 degrees
- moved D5 26.9 mm to (226.0, 135.4), turned to 90 degrees
- moved J1 25.8 mm to (221.4, 117.2), turned to 0 degrees
- moved R3 25.1 mm to (235.5, 123.6), turned to -90 degrees
- moved R7 24.8 mm to (221.4, 135.4)
- moved D1 24.8 mm to (221.4, 135.4)
- moved R2 23.9 mm to (237.0, 123.6), turned to -90 degrees
- moved R6 23.7 mm to (226.1, 132.2), turned to 180 degrees
- moved C2 18.3 mm to (234.0, 123.6), turned to 90 degrees
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- renumbered D3 to D2, D1 to D3, H2 to H1, H1 to H2, J2 to J1, J1 to J2, R6 to R2, R5 to R3, R7 to R4, R4 to R5, R2 to R6, R3 to R7
Routing:
- net Net-(U3-MGL): track 7.45 -> 22.6 mm, vias 2 -> 1
- net /MOSI: track 23.0 -> 8.54 mm, vias 1 -> 0
- net /CS: track 22.3 -> 8.47 mm
- net Net-(D2-A): track 2.99 -> 15.7 mm
- net Net-(U3-MGH): track 11.3 -> 20.3 mm, vias 1 -> 2
- net /B: track 5.32 -> 14.0 mm
- net /PWM: track 5.42 -> 12.4 mm
- net GND: track 22.2 -> 16.8 mm, vias 7 -> 11
- net Net-(R1-Pad1): track 8.02 -> 2.86 mm
- net Net-(U3-A): track 6.71 -> 1.92 mm
- net Net-(U3-B): track 5.53 -> 9.76 mm
- net +5V: track 5.59 -> 8.26 mm, vias 0 -> 1
- net Net-(D4-A): track 3.91 -> 5.65 mm
- net Net-(D5-A): track 2.72 -> 4.43 mm
- net +5V_IN: track 12.6 -> 14.2 mm
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Other:
- board size 26.7 x 31.8 mm -> 21.8 x 31.8 mm
- board text added: "1-GND 2-5V 3-A 4-B 5-PWM"
- board text added: "MAG ENCODER V1 971 SPARTAN ROBOTICS 2024"
- board text removed: "5-PWM 4-B 3-A 2-5V 1-GND"
- board text removed: "971 SPARTAN ROBOTICS 2024 MAG ENCODER V1"
