File: circuit-boards/shaft-encoders/mag-encoder/mag-encoder.kicad_sch (KiCad schematic)
At the start: 20 parts, among them J1 0015912055, U1 AP2120N-3.3TRG1, U2 SN74LVC1G02DBVR, U3 MA732GQ

Commit message: Add SPI header for config. Center mounting holes on sensor
Signed-off-by: Scott <sgberman1@gmail.com>
Parts:
- added H3: Pin, mag-encoder:pin-0.100, symbol Mechanical:MountingHole
- added H4: Slot, mag-encoder:slot-0.100x0.120, symbol Mechanical:MountingHole
- added J2: CONFIG, Connector_PinHeader_2.54mm:PinHeader_1x06_P2.54mm_Vertical, symbol Connector:Conn_01x06_Pin
Connections:
- net +3.3V: now also J2.2 (Pin_2)
- net GND: now also J2.1 (Pin_1)
- net SCLK: now reaches U3.12 (SCLK)
- net SCLK: now also J2.6 (Pin_6)
- net MOSI: now reaches U3.4 (MOSI)
- net MOSI: now also J2.4 (Pin_4)
- net CS: now reaches U3.5 (CS)
- net CS: now also J2.3 (Pin_3)
- net MISO: now reaches U3.7 (MISO)
- net MISO: now also J2.5 (Pin_5)
- no-connect marks 8 -> 4

Commit message: checkin of mag encoder
Signed-off-by: Scott <sgberman1@gmail.com>
Parts:
- removed H4: Slot, mag-encoder:slot-0.100x0.120, symbol Mechanical:MountingHole
- added C1: 1uF-10%-25V-0603, Capacitor_SMD:C_0603_1608Metric, symbol Device:C
- added H2: Slot, mag-encoder:pin-0.100, symbol Mechanical:MountingHole
- D2: renamed from D4; value HIGH -> HI
- D3: renamed from D2; value LOW -> LO
- D5: value PWR -> ON
- renumbered C1 to C3, D3 to D4, H2 to H1, H1 to H4, J2 to J1, J1 to J2, R6 to R2, R5 to R3, R7 to R4, R4 to R5, R2 to R6, R3 to R7, U2 to U1, U1 to U2
Connections:
- net +3.3V: now also C1.1
- net GND: now also C1.2
Other:
- moved on the sheet: H1, H4

Commit message: changed pins to 0.125".  Changed OK LED driver to mosfet.
Signed-off-by: Scott <sgberman1@gmail.com>
Parts:
- removed U1: SN74LVC1G02DBVR, Package_TO_SOT_SMD:SOT-23-5, symbol 74xGxx:74AUP1G02
- added Q1: BSS84, Package_TO_SOT_SMD:SOT-23, symbol Simulation_SPICE:PMOS
- renumbered D4 to D2, D2 to D3, D3 to D4, R2 to R1, R3 to R2, R4 to R3, R5 to R4, R6 to R5, R1 to R6, U2 to U1, U3 to U2
Connections:
- net +3.3V: now also Q1.2 (S)
- net GND: no longer D2.1 (K)
- net at R5.1, U2.16 (MGH): now also D2.1 (K)
- net at R6.1: now also Q1.3 (D)
- net at R4.1, U2.11 (MGL): now also Q1.1 (G)
Other:
- note removed: "Place LEDs connector side in incrementing order: LOW, OK, HIGH"
- moved on the sheet: R6
