File: circuit-boards/connector_boards/PowerDistribution-V2/PowerDistribution.kicad_pcb (KiCad board)
At the start: 2 copper layers, 70.5 x 76.2 mm, 27 parts, among them J1 2606-1102, J2 2604-1110, J3 2606-1102

Commit message: Export files for new pcbs + board characteristics
Signed-off-by: Alex lenkov <Alexander.i.lenkov@gmail.com>
Parts:
- removed the G*** at (160.8, 70.9)
- removed the G*** at (161.0, 136.7)
- moved F2 48.4 mm to (172.5, 114.4)
- moved F4 48.4 mm to (172.5, 94.4)
- moved D1 48.4 mm to (205.2, 81.9)
- moved D2 48.4 mm to (205.2, 91.9)
- moved D3 48.4 mm to (205.2, 101.9)
- moved D4 48.4 mm to (205.2, 111.9)
- moved D5 48.4 mm to (205.2, 121.9)
- moved F1 48.4 mm to (172.5, 124.4)
- moved G*** 48.4 mm to (177.9, 135.1)
- moved G*** 48.4 mm to (177.9, 69.0)
- moved H2 48.4 mm to (203.3, 133.8)
- moved H5 48.4 mm to (203.3, 70.3)
- moved J2 48.4 mm to (184.2, 124.4)
- moved R1 48.4 mm to (205.2, 76.9)
- moved R2 48.4 mm to (205.2, 86.9)
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Other:
- outline, holes or cut-outs redrawn
- board text added: "0"
- board text added: "0 mils"
- board text added: "0.0000 mm / 0.0000 mm"
- board text added: "0.02"
- board text added: "0.3000 mm"
- board text added: "0.3937 mils"
- board text added: "1"
- board text added: "1 oz"
- board text added: "1.37795 mils"
- board text added: "1.6000 mm"
- board text added: "1.Layers: 2 2.Thickness: 1.6 3.Surface finish: HASL 4.Outer Copper Weight: 2oz 5.Via covering: Tented 6.Min hole size: .3mm 7.Gold Fingers: No 8.Castellated Holes: No 9.Edge Plating: No"
- board text added: "2"
- board text added: "3.3"
- board text added: "4.5"
- board text added: "59.44882 mils"
- board text added: "70.4850 mm x 76.2000 mm"
- board text added: "B.Cu"
- board text added: "B.Mask"
- board text added: "B.Paste"
- board text added: "B.Silk"
- board text added: "B.Silkscreen"
- board text added: "BOARD CHARACTERISTICS"
- board text added: "Board Thickness:"
- board text added: "Board overall dimensions:"
- board text added: "Bottom Silk Screen"
- board text added: "Bottom Solder Mask"
- board text added: "Bottom Solder Paste"
- board text added: "Castellated pads:"
- board text added: "Color"
- board text added: "Copper Finish:"
- board text added: "Copper Layer Count:"
- board text added: "Dielectric"
- board text added: "Edge card connectors:"
- board text added: "Edge.Cuts"
- board text added: "Epsilon R"
- board text added: "F.Cu"
- board text added: "F.Mask"
- board text added: "F.Paste"
- board text added: "F.Silk"
- board text added: "F.Silkscreen"
- board text added: "FR4"
- board text added: "Impedance Control:"
- board text added: "LAYERS"
- board text added: "Layer Name"
- board text added: "Loss Tangent"
- board text added: "Margin"
- board text added: "Material"
- board text added: "Min hole diameter:"
- board text added: "Min track/spacing:"
- board text added: "NOTES"
- board text added: "No"
- board text added: "None"
- board text added: "Not specified"
- board text added: "Outer Copper Weight"
- board text added: "Plated Board Edge:"
- board text added: "Tented"
- board text added: "Thickness (mils)"
- board text added: "Top Silk Screen"
- board text added: "Top Solder Mask"
- board text added: "Top Solder Paste"
- board text added: "Type"
- board text added: "User.1"
- board text added: "Via Covering"
- board text added: "copper"
- board text added: "core"
- board text removed: "1.6mm 2 Ounce"

Commit message: Fix pcb fab layers
Signed-off-by: Alex lenkov <Alexander.i.lenkov@gmail.com>
Parts:
- removed REF**: Symbol_HighVoltage_Triangle_8x7mm_Copper, Symbol:Symbol_HighVoltage_Triangle_8x7mm_Copper
- moved H5 40.7 mm to (236.7, 47.0)
- moved H2 40.7 mm to (236.7, 110.5)
- moved G*** 38.1 mm to (208.2, 45.8)
- moved D1 37.2 mm to (234.1, 58.6)
- moved D2 37.2 mm to (234.1, 68.6)
- moved D5 37.2 mm to (234.2, 98.6)
- moved F3 37.2 mm to (201.3, 81.1)
- moved F5 37.2 mm to (201.4, 61.1)
- moved J1 37.2 mm to (183.3, 92.1)
- moved J3 37.2 mm to (183.3, 66.7)
- moved R4 37.2 mm to (234.2, 83.6)
- moved R5 37.2 mm to (234.2, 93.6)
- moved G*** 37.2 mm to (206.8, 111.8)
- moved R1 37.2 mm to (234.2, 53.6)
- moved R2 37.2 mm to (234.2, 63.6)
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Routing:
- net -BATT: track 31.5 -> 0.00 mm
- net +BATT: track 31.5 -> 0.00 mm
Other:
- outline, holes or cut-outs redrawn
- board text added: "2024"
- board text added: "FRONT"
- board text removed: "1 oz"
- board text removed: "Outer Copper Weight"
- board text removed: "Tented"
- board text removed: "Via Covering"
