File: circuit-boards/connector_boards/PowerDistribution-V2/PowerDistribution.kicad_pcb (KiCad board)
At the start: 2 copper layers, 70.5 x 76.2 mm, 24 parts, among them J1 2606-1102, J2 2604-1110, J3 2606-1102

Commit message: Add thermal relief for resistors
Signed-off-by: scott <sgberman1@gmail.com>
Routing:
- net -BATT: track 0.00 -> 41.0 mm
Changed lines of the file:
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@@
+	)
+	(segment
+		(start 213.093371 66.083471)
+		(end 221.29337 66.083471)
+		(width 3.429)
+		(layer "F.Cu")
+		(net 10)
+	)
+	(segment
+		(start 213.093371 76.083471)
+		(end 221.29337 76.083471)
+		(width 3.429)
+		(layer "F.Cu")
+		(net 10)
+	)
+	(segment
+		(start 213.093371 56.08347)
+		(end 221.29337 56.08347)
+		(width 3.429)
+		(layer "F.Cu")
+		(net 10)
+	)
+	(segment
+		(start 213.093371 96.083472)
+		(end 221.29337 96.083472)
+		(width 3.429)
+		(layer "F.Cu")
+		(net 10)
+	)
+	(segment
+		(start 213.093371 86.083471)
+		(end 221.29337 86.083471)
+		(width 3.429)
+		(layer "F.Cu")
+		(net 10)
 	)
 	(segment
@@
 		(layer "F.Cu")
 		(hatch edge 0.5)
-		(connect_pads yes
+		(connect_pads
 			(clearance 0.508)
 		)
@@
 		(filled_areas_thickness no)
 		(fill yes
-			(thermal_gap 0.635)
-			(thermal_bridge_width 1.016)
+			(thermal_gap 0.381)
+			(thermal_bridge_width 0.254)
 		)
 		(polygon
