File: circuit-boards/hall-switch-v2/HallSwitch.kicad_sch (KiCad schematic)
At the start: 12 parts, among them J1 0705550037, U1 US5881ESE

Commit message: Fix pcb fab layers
Signed-off-by: Alex lenkov <Alexander.i.lenkov@gmail.com>
Other:
- company: Spartan Robotics -> 971 SPARTAN ROBOTICS
Changed lines of the file:
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@@
 	(title_block
 		(title "Hall Switch")
-		(date "2024-08-30")
+		(date "2024-10-12")
 		(rev "R2")
-		(company "Spartan Robotics")
+		(company "971 SPARTAN ROBOTICS")
 	)
 	(junction
